File: Hardware/Schematics/BBDProto03/BBDProto03.kicad_pcb (KiCad board)
At the start: 2 copper layers, 68.6 x 53.3 mm, 8 parts, among them P1 Power, P2 Analog, P3 Digital, P4 Digital, P5 CONN_1, P6 CONN_1, P7 CONN_1, P8 CONN_1

Commit message: Library updates, photos, FreeRoute
Library updates, photos, FreeRoute
Parts:
- added C1: 100nF, Capacitors_SMD:C_0603_HandSoldering, F.Cu at (128.8, 111.1)
- added Cin1: 100nF, Capacitors_SMD:C_0603_HandSoldering, F.Cu at (141.5, 116.2)
- added Cout1: 100nF, Capacitors_SMD:C_0603_HandSoldering, F.Cu at (141.5, 111.1)
- added L1: 1uH, Inductors:NR4018_HandSoldering, F.Cu at (118.6, 117.5)
- added P11: CONN_02X08, Socket_Strips:Socket_Strip_Straight_2x08, F.Cu at (205.0, 118.7)
- added P12: CONN_02X08, Socket_Strips:Socket_Strip_Straight_2x08, F.Cu at (213.9, 141.6)
- added P13: CONN_02X08, Socket_Strips:Socket_Strip_Straight_2x08, F.Cu at (207.5, 78.1)
- added R1: 1.2k, Resistors_SMD:R_0603_HandSoldering, F.Cu at (128.8, 116.2)
- added R2: 10m, Resistors_SMD:R_0603_HandSoldering, F.Cu at (135.1, 111.1)
- added R3: 10m, Resistors_SMD:R_0603_HandSoldering, F.Cu at (152.9, 90.8)
- added U1: ATTINY861-20SU, Housings_SOIC:SOIC-20_7.5x12.8mm_Pitch1.27mm, F.Cu at (135.1, 90.8)
- added U10: CD74HC4067, Housings_SSOP:SSOP-24_5.3x8.2mm_Pitch0.65mm, F.Cu at (164.3, 106.0)
- added U11: CD74HC4067, Housings_SSOP:SSOP-24_5.3x8.2mm_Pitch0.65mm, F.Cu at (189.7, 112.4)
- added U12: CD74HC4067, Housings_SSOP:SSOP-24_5.3x8.2mm_Pitch0.65mm, F.Cu at (198.6, 140.3)
- added U13: CD74HC4067, Housings_SSOP:SSOP-24_5.3x8.2mm_Pitch0.65mm, F.Cu at (189.7, 87.0)
- added U2: LTC1864, Housings_SOIC:SOIC-8_3.9x4.9mm_Pitch1.27mm, F.Cu at (151.6, 103.5)
- added U3: LTC3407, Housings_SSOP:MSOP-10-1EP_3x3mm_Pitch0.5mm, F.Cu at (118.6, 90.8)
- added U4: MCP4161, Housings_SOIC:SOIC-8_3.9x4.9mm_Pitch1.27mm, F.Cu at (119.9, 104.8)
Connections:
- P1 pad 4: +3V3 -> /+3.3V
- P1 pad 5: +5V -> /+5.0V
- P2 pad 5: /A4(SDA) -> /+5.0V
- P2 pad 6: /A5(SCL) -> /+3.3V
- P3 pad 1: /A5(SCL) -> /+3.3V
- P3 pad 2: /A4(SDA) -> /+5.0V
