File: Hardware/Schematics/BBDProto06/Venus-256/Venus-256.sch (KiCad schematic (older format))
At the start: 1 part, among them U1 ADG715

Commit message: Updated the AD7616 and its Cell Slave schematics
Updated the AD7616 and its Cell Slave schematics
Parts:
- U101: renamed from U1; symbol Analog:ADG715 -> Analog_Switch:ADG715
Connections:
- wire segments 242 -> 238
Changed lines of the file:
@@
 $EndSheet
 $Comp
-L power:GND #PWR07
+L power:GND #PWR0106
 U 1 1 5AE8F6FC
 P 4100 3300
-F 0 "#PWR07" H 4100 3050 50  0001 C CNN
+F 0 "#PWR0106" H 4100 3050 50  0001 C CNN
 F 1 "GND" H 4105 3127 50  0000 C CNN
 F 2 "" H 4100 3300 50  0001 C CNN
@@
 	4100 3100 4100 3300
 $Comp
-L power:GND #PWR02
+L power:GND #PWR0103
 U 1 1 5AE8F71C
 P 1000 3000
-F 0 "#PWR02" H 1000 2750 50  0001 C CNN
+F 0 "#PWR0103" H 1000 2750 50  0001 C CNN
 F 1 "GND" H 1005 2827 50  0000 C CNN
 F 2 "" H 1000 3000 50  0001 C CNN
@@
 	1000 2800 1000 3000
 $Comp
-L power:GND #PWR01
+L power:GND #PWR0102
 U 1 1 5AE8F730
 P 1000 1500
-F 0 "#PWR01" H 1000 1250 50  0001 C CNN
+F 0 "#PWR0102" H 1000 1250 50  0001 C CNN
 F 1 "GND" H 1005 1327 50  0000 C CNN
 F 2 "" H 1000 1500 50  0001 C CNN
@@
 Connection ~ 800  1000
 $Comp
-L power:GND #PWR09
+L power:GND #PWR0108
 U 1 1 5AE90A11
 P 9900 1600
-F 0 "#PWR09" H 9900 1350 50  0001 C CNN
+F 0 "#PWR0108" H 9900 1350 50  0001 C CNN
 F 1 "GND" H 9905 1427 50  0000 C CNN
 F 2 "" H 9900 1600 50  0001 C CNN
@@
 	9900 1400 9900 1600
 $Comp
-L power:GND #PWR013
+L power:GND #PWR0113
 U 1 1 5AE919C7
 P 10100 1600
-F 0 "#PWR013" H 10100 1350 50  0001 C CNN
+F 0 "#PWR0113" H 10100 1350 50  0001 C CNN
 F 1 "GND" H 10105 1427 50  0000 C CNN
 F 2 "" H 10100 1600 50  0001 C CNN
@@
 	10400 2300 9800 2300
 $Comp
-L power:GND #PWR010
+L power:GND #PWR0109
 U 1 1 5AE958F1
 P 9900 2900
-F 0 "#PWR010" H 9900 2650 50  0001 C CNN
+F 0 "#PWR0109" H 9900 2650 50  0001 C CNN
 F 1 "GND" H 9905 2727 50  0000 C CNN
 F 2 "" H 9900 2900 50  0001 C CNN
@@
 	9900 2700 9900 2900
 $Comp
-L power:GND #PWR014
+L power:GND #PWR0114
 U 1 1 5AE958F9
 P 10100 2900
-F 0 "#PWR014" H 10100 2650 50  0001 C CNN
+F 0 "#PWR0114" H 10100 2650 50  0001 C CNN
 F 1 "GND" H 10105 2727 50  0000 C CNN
 F 2 "" H 10100 2900 50  0001 C CNN
@@
 	10400 3600 9800 3600
 $Comp
-L power:GND #PWR011
+L power:GND #PWR0110
 U 1 1 5AE96319
 P 9900 4200
-F 0 "#PWR011" H 9900 3950 50  0001 C CNN
+F 0 "#PWR0110" H 9900 3950 50  0001 C CNN
 F 1 "GND" H 9905 4027 50  0000 C CNN
 F 2 "" H 9900 4200 50  0001 C CNN
@@
 	9900 4000 9900 4200
 $Comp
-L power:GND #PWR015
+L power:GND #PWR0115
 U 1 1 5AE96321
 P 10100 4200
-F 0 "#PWR015" H 10100 3950 50  0001 C CNN
+F 0 "#PWR0115" H 10100 3950 50  0001 C CNN
 F 1 "GND" H 10105 4027 50  0000 C CNN
 F 2 "" H 10100 4200 50  0001 C CNN
@@
 	10400 4900 9800 4900
 $Comp
-L power:GND #PWR012
+L power:GND #PWR0111
 U 1 1 5AE96EDB
 P 9900 5500
-F 0 "#PWR012" H 9900 5250 50  0001 C CNN
+F 0 "#PWR0111" H 9900 5250 50  0001 C CNN
 F 1 "GND" H 9905 5327 50  0000 C CNN
 F 2 "" H 9900 5500 50  0001 C CNN
@@
 	9900 5300 9900 5500
 $Comp
-L power:GND #PWR016
+L power:GND #PWR0116
 U 1 1 5AE96EE3
 P 10100 5500
-F 0 "#PWR016" H 10100 5250 50  0001 C CNN
+F 0 "#PWR0116" H 10100 5250 50  0001 C CNN
 F 1 "GND" H 10105 5327 50  0000 C CNN
 F 2 "" H 10100 5500 50  0001 C CNN
@@
 	2800 1300 3500 1300
 $Comp
-L Analog:ADG715 U1
-U 1 1 5AE36C1A
-P 1800 4600
-F 0 "U1" H 1300 5200 50  0000 C CNN
-F 1 "ADG715" H 1400 4100 50  0000 C CNN
-F 2 "Package_SO:TSSOP-24_4.4x7.8mm_P0.65mm" H 2800 4100 50  0001 C CIN
-F 3 "http://www.analog.com/media/en/technical-documentation/data-sheets/ADG714_715.pdf" H 1800 4400 50  0001 C CNN
-	1    1800 4600
+L power:GND #PWR0104
+U 1 1 5AE36CCF
+P 1700 6250
+F 0 "#PWR0104" H 1700 6000 50  0001 C CNN
+F 1 "GND" H 1705 6077 50  0000 C CNN
+F 2 "" H 1700 6250 50  0001 C CNN
+F 3 "" H 1700 6250 50  0001 C CNN
+	1    1700 6250
 	1    0    0    -1
 $EndComp
-$Comp
-L power:GND #PWR04
-U 1 1 5AE36CCF
-P 2000 5500
-F 0 "#PWR04" H 2000 5250 50  0001 C CNN
-F 1 "GND" H 2005 5327 50  0000 C CNN
-F 2 "" H 2000 5500 50  0001 C CNN
-F 3 "" H 2000 5500 50  0001 C CNN
-	1    2000 5500
-	1    0    0    -1
-$EndComp
 Wire Wire Line
 	4200 1100 4100 1100
@@
 	4100 1100 4100 1000
 Wire Wire Line
-	3000 1000 3000 4200
-Wire Wire Line
-	3000 4200 2500 4200
+	3000 1000 3000 4400
 Wire Wire Line
 	3000 1000 4100 1000
@@
 Connection ~ 4100 1000
 Wire Wire Line
-	800  2200 800  3600
-Wire Wire Line
-	800  4900 1100 4900
+	800  2200 800  3800
 Connection ~ 800  2200
 Wire Wire Line
-	800  4800 1100 4800
-Connection ~ 800  4800
-Wire Wire Line
-	800  4800 800  4900
-Wire Wire Line
-	800  4200 1100 4200
-Connection ~ 800  4200
-Wire Wire Line
-	800  4200 800  4300
-Wire Wire Line
-	1100 4300 800  4300
-Connection ~ 800  4300
-Wire Wire Line
-	800  4300 800  4400
-Wire Wire Line
-	800  4400 1100 4400
-Connection ~ 800  4400
-Wire Wire Line
-	800  4400 800  4500
-Wire Wire Line
-	1100 4500 800  4500
-Connection ~ 800  4500
-Wire Wire Line
-	800  4500 800  4600
-Wire Wire Line
-	800  4600 1100 4600
-Connection ~ 800  4600
-Wire Wire Line
-	800  4600 800  4700
-Wire Wire Line
-	1100 4700 800  4700
-Connection ~ 800  4700
-Wire Wire Line
-	800  4700 800  4800
-Wire Wire Line
-	2000 5200 2000 5500
-$Comp
-L power:GND #PWR03
+	1700 5900 1700 6250
+$Comp
+L power:GND #PWR0105
 U 1 1 5AE90B6E
-P 1900 5300
-F 0 "#PWR03" H 1900 5050 50  0001 C CNN
-F 1 "GND" H 1905 5127 50  0000 C CNN
-F 2 "" H 1900 5300 50  0001 C CNN
-F 3 "" H 1900 5300 50  0001 C CNN
-	1    1900 5300
+P 1900 6250
+F 0 "#PWR0105" H 1900 6000 50  0001 C CNN
+F 1 "GND" H 1905 6077 50  0000 C CNN
+F 2 "" H 1900 6250 50  0001 C CNN
+F 3 "" H 1900 6250 50  0001 C CNN
+	1    1900 6250
 	1    0    0    -1
 $EndComp
 Wire Wire Line
-	1900 5200 1900 5300
-Wire Wire Line
 	1100 2500 600  2500
 Wire Wire Line
-	600  2500 600  5500
-Wire Wire Line
-	600  5500 1600 5500
-Wire Wire Line
-	1600 5500 1600 5200
+	600  2500 600  5400
 Wire Wire Line
 	1100 2600 700  2600
-Wire Wire Line
-	700  2600 700  5400
-Wire Wire Line
-	700  5400 1700 5400
-Wire Wire Line
-	1700 5400 1700 5200
-Wire Wire Line
-	2100 3900 2100 3600
-Wire Wire Line
-	2100 3600 2300 3600
-Wire Wire Line
-	2300 3600 2300 3700
-$Comp
-L power:GND #PWR06
+$Comp
+L power:GND #PWR0101
 U 1 1 5AEC21F3
-P 2300 3700
-F 0 "#PWR06" H 2300 3450 50  0001 C CNN
-F 1 "GND" H 2305 3527 50  0000 C CNN
-F 2 "" H 2300 3700 50  0001 C CNN
-F 3 "" H 2300 3700 50  0001 C CNN
-	1    2300 3700
+P 700 6250
+F 0 "#PWR0101" H 700 6000 50  0001 C CNN
+F 1 "GND" H 705 6077 50  0000 C CNN
+F 2 "" H 700 6250 50  0001 C CNN
+F 3 "" H 700 6250 50  0001 C CNN
+	1    700  6250
 	1    0    0    -1
 $EndComp
 Wire Wire Line
-	1900 3900 1900 3200
-Wire Wire Line
-	1900 3200 2100 3200
-Wire Wire Line
-	2100 3200 2100 3300
-$Comp
-L power:GND #PWR05
-U 1 1 5AECD1C2
-P 2100 3300
-F 0 "#PWR05" H 2100 3050 50  0001 C CNN
-F 1 "GND" H 2105 3127 50  0000 C CNN
-F 2 "" H 2100 3300 50  0001 C CNN
-F 3 "" H 2100 3300 50  0001 C CNN
-	1    2100 3300
-	1    0    0    -1
-$EndComp
-Wire Wire Line
-	800  3600 1500 3600
-Wire Wire Line
-	1700 3600 1700 3900
-Connection ~ 800  3600
-Wire Wire Line
-	800  3600 800  4200
-Wire Wire Line
-	1500 3600 1500 3900
-Connection ~ 1500 3600
-Wire Wire Line
-	1500 3600 1700 3600
+	1800 3800 1800 4100
 $Sheet
 S 4200 6550 1300 2300
@@
 $EndSheet
 $Comp
-L power:GND #PWR08
+L power:GND #PWR0107
 U 1 1 5AF03082
 P 4100 8950
-F 0 "#PWR08" H 4100 8700 50  0001 C CNN
+F 0 "#PWR0107" H 4100 8700 50  0001 C CNN
 F 1 "GND" H 4105 8777 50  0000 C CNN
 F 2 "" H 4100 8950 50  0001 C CNN
@@
 	3200 1600 4200 1600
 Wire Wire Line
-	2500 4300 3000 4300
-Wire Wire Line
-	3000 4300 3000 6650
+	3000 4500 3000 6650
 Wire Wire Line
 	3000 6650 4100 6650
@@
 	8000 7550 8500 7550
 $Comp
-L power:GND #PWR0101
+L power:GND #PWR0112
 U 1 1 5B09A94C
 P 9900 7250
-F 0 "#PWR0101" H 9900 7000 50  0001 C CNN
+F 0 "#PWR0112" H 9900 7000 50  0001 C CNN
 F 1 "GND" H 9905 7077 50  0000 C CNN
 F 2 "" H 9900 7250 50  0001 C CNN
@@
 	9900 7050 9900 7250
 $Comp
-L power:GND #PWR0102
+L power:GND #PWR0117
 U 1 1 5B09A954
 P 10100 7250
-F 0 "#PWR0102" H 10100 7000 50  0001 C CNN
+F 0 "#PWR0117" H 10100 7000 50  0001 C CNN
 F 1 "GND" H 10105 7077 50  0000 C CNN
 F 2 "" H 10100 7250 50  0001 C CNN
@@
 Wire Wire Line
 	9800 6950 10300 6950
+$Comp
+L Analog_Switch:ADG715 U101
+U 1 1 5AE36C1A
+P 1800 5100
+F 0 "U101" H 1150 6050 50  0000 C CNN
+F 1 "ADG715" H 2350 6050 50  0000 C CNN
+F 2 "Package_SO:TSSOP-24_4.4x7.8mm_P0.65mm" H 2800 4600 50  0001 C CIN
+F 3 "http://www.analog.com/media/en/technical-documentation/data-sheets/ADG714_715.pdf" H 1800 4900 50  0001 C CNN
+	1    1800 5100
+	1    0    0    -1
+$EndComp
+Wire Wire Line
+	1900 5900 1900 6250
+Wire Wire Line
+	800  3800 1800 3800
+Wire Wire Line
+	800  3800 800  4400
+Wire Wire Line
+	800  5300 1000 5300
+Connection ~ 800  3800
+Wire Wire Line
+	1000 5500 700  5500
+Wire Wire Line
+	700  2600 700  5500
+Wire Wire Line
+	600  5400 1000 5400
+Wire Wire Line
+	700  5600 700  5700
+Wire Wire Line
+	700  5600 1000 5600
+Wire Wire Line
+	1000 5700 700  5700
+Connection ~ 700  5700
+Wire Wire Line
+	700  5700 700  6250
+Wire Wire Line
+	3000 4500 2600 4500
+Wire Wire Line
+	2600 4400 3000 4400
+Wire Wire Line
+	800  4400 1000 4400
+Connection ~ 800  4400
+Wire Wire Line
+	800  4400 800  4500
+Wire Wire Line
+	800  4500 1000 4500
+Connection ~ 800  4500
+Wire Wire Line
+	800  4500 800  4600
+Wire Wire Line
+	800  4600 1000 4600
+Connection ~ 800  4600
+Wire Wire Line
+	800  4600 800  4700
+Wire Wire Line
+	800  4700 1000 4700
+Connection ~ 800  4700
+Wire Wire Line
+	800  4700 800  4800
+Wire Wire Line
+	800  4800 1000 4800
+Connection ~ 800  4800
+Wire Wire Line
+	800  4800 800  4900
+Wire Wire Line
+	800  4900 1000 4900
+Connection ~ 800  4900
+Wire Wire Line
+	800  4900 800  5000
+Wire Wire Line
+	800  5000 1000 5000
+Connection ~ 800  5000
+Wire Wire Line
+	800  5000 800  5100
+Wire Wire Line
+	800  5100 1000 5100
+Connection ~ 800  5100
+Wire Wire Line
+	800  5100 800  5300
 $EndSCHEMATC
