File: Hardware/Schematics/BBDProto06/Venus-256/Venus-256.sch (KiCad schematic (older format))
At the start: 1 part, among them U101 ADG715

Commit message: Fixed many rules check errors and changed the footprint of test points
Connections:
- wire segments 238 -> 249
- no-connect marks 0 -> 17
Changed lines of the file:
@@
 	1800 3800 1800 4100
 $Sheet
-S 4200 6550 1300 2300
+S 4200 6500 1300 2300
 U 5AF0307C
 F0 "CellMaster-02" 50
 F1 "CellMaster.sch" 50
-F2 "VCC_MCU_P3V3" I L 4200 6650 50
-F3 "VDDCORE" I L 4200 6750 50
-F4 "GND" I L 4200 8750 50
-F5 "TRACESWO" O L 4200 6950 50
-F6 "SWDIO" B L 4200 7050 50
-F7 "SWCLK" I L 4200 7150 50
-F8 "TARGET_RESET" I L 4200 7250 50
-F9 "SPI1_NPCS0" O R 5500 7150 50
-F10 "SPI0_MISO" O L 4200 7450 50
-F11 "SPI0_MOSI" I L 4200 7550 50
-F12 "SPI0_SPCK" I L 4200 7650 50
-F13 "SPI1_NPCS2" O R 5500 7950 50
-F14 "SPI1_NPCS1" O R 5500 7550 50
-F15 "DAC0" O R 5500 6750 50
-F16 "SPI1_NPCS3" O R 5500 8350 50
-F17 "SPI1_MISO" I R 5500 8550 50
-F18 "SPI1_MOSI" O R 5500 8650 50
-F19 "SPI1_SPCK" O R 5500 8750 50
-F20 "ADC_CONVST0" O R 5500 6950 50
-F21 "ADC_BUSY0" I R 5500 7050 50
-F22 "ADC_BUSY1" I R 5500 7450 50
-F23 "ADC_BUSY2" I R 5500 7850 50
-F24 "ADC_BUSY3" I R 5500 8250 50
-F25 "ADC_CONVST1" O R 5500 7350 50
-F26 "ADC_CONVST2" O R 5500 7750 50
-F27 "ADC_CONVST3" O R 5500 8150 50
-F28 "ADC_RESET" I R 5500 6650 50
+F2 "VCC_MCU_P3V3" I L 4200 6600 50
+F3 "VDDCORE" I L 4200 6700 50
+F4 "GND" I L 4200 8700 50
+F5 "TRACESWO" O L 4200 6900 50
+F6 "SWDIO" B L 4200 7000 50
+F7 "SWCLK" I L 4200 7100 50
+F8 "TARGET_RESET" I L 4200 7200 50
+F9 "SPI1_NPCS0" O R 5500 7100 50
+F10 "SPI0_MISO" O L 4200 7400 50
+F11 "SPI0_MOSI" I L 4200 7500 50
+F12 "SPI0_SPCK" I L 4200 7600 50
+F13 "SPI1_NPCS2" O R 5500 7900 50
+F14 "SPI1_NPCS1" O R 5500 7500 50
+F15 "DAC0" O R 5500 6700 50
+F16 "SPI1_NPCS3" O R 5500 8300 50
+F17 "SPI1_MISO" I R 5500 8500 50
+F18 "SPI1_MOSI" O R 5500 8600 50
+F19 "SPI1_SPCK" O R 5500 8700 50
+F20 "ADC_CONVST0" O R 5500 6900 50
+F21 "ADC_BUSY0" I R 5500 7000 50
+F22 "ADC_BUSY1" I R 5500 7400 50
+F23 "ADC_BUSY2" I R 5500 7800 50
+F24 "ADC_BUSY3" I R 5500 8200 50
+F25 "ADC_CONVST1" O R 5500 7300 50
+F26 "ADC_CONVST2" O R 5500 7700 50
+F27 "ADC_CONVST3" O R 5500 8100 50
+F28 "ADC_RESET" I R 5500 6600 50
 $EndSheet
 $Comp
@@
 $EndComp
 Wire Wire Line
-	4200 8750 4100 8750
-Wire Wire Line
-	4100 8750 4100 8950
-Wire Wire Line
-	4200 7450 3900 7450
-Wire Wire Line
-	4200 6750 4100 6750
-Wire Wire Line
-	4100 6750 4100 6650
-Wire Wire Line
-	4200 6650 4100 6650
-Wire Wire Line
-	3900 7450 3900 1800
+	4200 8700 4100 8700
+Wire Wire Line
+	4100 8700 4100 8950
+Wire Wire Line
+	4200 7400 3900 7400
+Wire Wire Line
+	4200 6700 4100 6700
+Wire Wire Line
+	4100 6700 4100 6600
+Wire Wire Line
+	4200 6600 4100 6600
+Wire Wire Line
+	3900 7400 3900 1800
 Connection ~ 3900 1800
 Wire Wire Line
 	3900 1800 2500 1800
 Wire Wire Line
-	3800 7550 3800 1900
-Wire Wire Line
-	3800 7550 4200 7550
+	3800 7500 3800 1900
+Wire Wire Line
+	3800 7500 4200 7500
 Connection ~ 3800 1900
 Wire Wire Line
 	3800 1900 2600 1900
 Wire Wire Line
-	3700 7650 3700 2000
-Wire Wire Line
-	3700 7650 4200 7650
+	3700 7600 3700 2000
+Wire Wire Line
+	3700 7600 4200 7600
 Connection ~ 3700 2000
 Wire Wire Line
 	3700 2000 2700 2000
 Wire Wire Line
-	4200 6950 3500 6950
-Wire Wire Line
-	3500 6950 3500 1300
+	4200 6900 3500 6900
+Wire Wire Line
+	3500 6900 3500 1300
 Connection ~ 3500 1300
 Wire Wire Line
 	3500 1300 4200 1300
 Wire Wire Line
-	4200 7050 3400 7050
-Wire Wire Line
-	3400 7050 3400 1400
+	4200 7000 3400 7000
+Wire Wire Line
+	3400 7000 3400 1400
 Connection ~ 3400 1400
 Wire Wire Line
 	3400 1400 4200 1400
 Wire Wire Line
-	4200 7150 3300 7150
-Wire Wire Line
-	3300 7150 3300 1500
+	4200 7100 3300 7100
+Wire Wire Line
+	3300 7100 3300 1500
 Connection ~ 3300 1500
 Wire Wire Line
 	3300 1500 4200 1500
 Wire Wire Line
-	4200 7250 3200 7250
-Wire Wire Line
-	3200 7250 3200 1600
+	4200 7200 3200 7200
+Wire Wire Line
+	3200 7200 3200 1600
 Connection ~ 3200 1600
 Wire Wire Line
 	3200 1600 4200 1600
 Wire Wire Line
-	3000 4500 3000 6650
-Wire Wire Line
-	3000 6650 4100 6650
-Connection ~ 4100 6650
+	3000 4500 3000 6600
+Wire Wire Line
+	3000 6600 4100 6600
+Connection ~ 4100 6600
 $Sheet
-S 8500 6550 1300 1100
+S 8500 6500 1300 1100
 U 5AFE7089
 F0 "CellSlave-02A" 50
 F1 "CellSlave.sch" 50
-F2 "DGND" U R 9800 7050 50
-F3 "BUSY" O L 8500 7050 50
-F4 "~CS" I L 8500 7150 50
-F5 "VDRIVE_3V3" I R 9800 6950 50
-F6 "SDI" I L 8500 7450 50
-F7 "SDOA" O L 8500 7350 50
-F8 "SCLK" I L 8500 7550 50
-F9 "AGND" U R 9800 6750 50
-F10 "VCC_5V0" I R 9800 6650 50
-F11 "SGND" I L 8500 6750 50
-F12 "~RESET" I L 8500 6650 50
-F13 "CONVST" I L 8500 6950 50
+F2 "DGND" U R 9800 7000 50
+F3 "BUSY" O L 8500 7000 50
+F4 "~CS" I L 8500 7100 50
+F5 "VDRIVE_3V3" I R 9800 6900 50
+F6 "SDI" I L 8500 7400 50
+F7 "SDOA" O L 8500 7300 50
+F8 "SCLK" I L 8500 7500 50
+F9 "AGND" U R 9800 6700 50
+F10 "VCC_5V0" I R 9800 6600 50
+F11 "SGND" I L 8500 6700 50
+F12 "~RESET" I L 8500 6600 50
+F13 "CONVST" I L 8500 6900 50
 $EndSheet
 Wire Wire Line
-	5500 6650 8500 6650
-Wire Wire Line
-	10300 5200 10300 6950
+	5500 6600 8500 6600
+Wire Wire Line
+	10300 5200 10300 6900
 Connection ~ 10300 5200
 Wire Wire Line
-	9800 6650 10400 6650
-Wire Wire Line
-	10400 6650 10400 4900
+	9800 6600 10400 6600
+Wire Wire Line
+	10400 6600 10400 4900
 Connection ~ 10400 4900
 Wire Wire Line
-	5500 6750 8500 6750
-Wire Wire Line
-	5500 6950 8500 6950
-Wire Wire Line
-	5500 7050 8500 7050
-Wire Wire Line
-	5500 7150 8500 7150
-Wire Wire Line
-	5500 8550 7800 8550
-Wire Wire Line
-	7800 8550 7800 7350
-Wire Wire Line
-	7800 7350 8500 7350
-Wire Wire Line
-	8500 7450 7900 7450
-Wire Wire Line
-	7900 7450 7900 8650
-Wire Wire Line
-	7900 8650 5500 8650
-Wire Wire Line
-	5500 8750 8000 8750
-Wire Wire Line
-	8000 8750 8000 7550
-Wire Wire Line
-	8000 7550 8500 7550
+	5500 6700 8500 6700
+Wire Wire Line
+	5500 6900 8500 6900
+Wire Wire Line
+	5500 7000 8500 7000
+Wire Wire Line
+	5500 7100 8500 7100
+Wire Wire Line
+	5500 8500 7800 8500
+Wire Wire Line
+	7800 8500 7800 7300
+Wire Wire Line
+	7800 7300 8500 7300
+Wire Wire Line
+	8500 7400 7900 7400
+Wire Wire Line
+	7900 7400 7900 8600
+Wire Wire Line
+	7900 8600 5500 8600
+Wire Wire Line
+	5500 8700 8000 8700
+Wire Wire Line
+	8000 8700 8000 7500
+Wire Wire Line
+	8000 7500 8500 7500
 $Comp
 L power:GND #PWR0112
@@
 $EndComp
 Wire Wire Line
-	9800 7050 9900 7050
-Wire Wire Line
-	9900 7050 9900 7250
+	9800 7000 9900 7000
+Wire Wire Line
+	9900 7000 9900 7250
 $Comp
 L power:GND #PWR0117
@@
 $EndComp
 Wire Wire Line
-	10100 6750 10100 7250
-Wire Wire Line
-	9800 6750 10100 6750
-Wire Wire Line
-	9800 6950 10300 6950
+	10100 6700 10100 7250
+Wire Wire Line
+	9800 6700 10100 6700
+Wire Wire Line
+	9800 6900 10300 6900
 $Comp
 L Analog_Switch:ADG715 U101
@@
 Wire Wire Line
 	800  5100 800  5300
+NoConn ~ 2600 4600
+NoConn ~ 2600 4700
+NoConn ~ 2600 4800
+NoConn ~ 2600 4900
+NoConn ~ 2600 5000
+NoConn ~ 2600 5100
+NoConn ~ 2500 2600
+NoConn ~ 2500 2700
+Wire Wire Line
+	2500 2600 2400 2600
+Wire Wire Line
+	2400 2700 2500 2700
+NoConn ~ 5600 7300
+NoConn ~ 5600 7400
+NoConn ~ 5600 7500
+NoConn ~ 5600 7700
+NoConn ~ 5600 7800
+NoConn ~ 5600 7900
+NoConn ~ 5600 8100
+NoConn ~ 5600 8200
+NoConn ~ 5600 8300
+Wire Wire Line
+	5500 7300 5600 7300
+Wire Wire Line
+	5500 7400 5600 7400
+Wire Wire Line
+	5500 7500 5600 7500
+Wire Wire Line
+	5500 7700 5600 7700
+Wire Wire Line
+	5500 7800 5600 7800
+Wire Wire Line
+	5500 7900 5600 7900
+Wire Wire Line
+	5500 8100 5600 8100
+Wire Wire Line
+	5500 8200 5600 8200
+Wire Wire Line
+	5500 8300 5600 8300
 $EndSCHEMATC

Commit message: Replaced the ADG715 with TPS22993
Parts:
- removed U101: ADG715, Package_SO:TSSOP-24_4.4x7.8mm_P0.65mm, symbol Analog_Switch:ADG715
- added TP101: VOUT3_TP, TestPoint:TestPoint_Pad_1.0x1.0mm, symbol Venus-256-rescue:Test_Point_Flag-Connector_Specialized
- added TP102: VOUT4_TP, TestPoint:TestPoint_Pad_1.0x1.0mm, symbol Venus-256-rescue:Test_Point_Flag-Connector_Specialized
- added U101: TPS22993, Package_DFN_QFN:Texas_S-PWQFN-N20, symbol Power_Management:TPS22993
Connections:
- wire segments 249 -> 258
- no-connect marks 17 -> 11
Changed lines of the file:
@@
 	800  2200 1100 2200
 Wire Wire Line
-	1100 2300 700  2300
+	1100 2300 900  2300
 Wire Wire Line
 	700  2300 700  600
@@
 L power:GND #PWR0104
 U 1 1 5AE36CCF
-P 1700 6250
-F 0 "#PWR0104" H 1700 6000 50  0001 C CNN
-F 1 "GND" H 1705 6077 50  0000 C CNN
-F 2 "" H 1700 6250 50  0001 C CNN
-F 3 "" H 1700 6250 50  0001 C CNN
-	1    1700 6250
+P 1500 6300
+F 0 "#PWR0104" H 1500 6050 50  0001 C CNN
+F 1 "GND" H 1505 6127 50  0000 C CNN
+F 2 "" H 1500 6300 50  0001 C CNN
+F 3 "" H 1500 6300 50  0001 C CNN
+	1    1500 6300
 	1    0    0    -1
 $EndComp
@@
 	4100 1100 4100 1000
 Wire Wire Line
-	3000 1000 3000 4400
+	3000 1000 3000 4800
 Wire Wire Line
 	3000 1000 4100 1000
@@
 Connection ~ 800  2200
 Wire Wire Line
-	1700 5900 1700 6250
-$Comp
-L power:GND #PWR0105
-U 1 1 5AE90B6E
-P 1900 6250
-F 0 "#PWR0105" H 1900 6000 50  0001 C CNN
-F 1 "GND" H 1905 6077 50  0000 C CNN
-F 2 "" H 1900 6250 50  0001 C CNN
-F 3 "" H 1900 6250 50  0001 C CNN
-	1    1900 6250
-	1    0    0    -1
-$EndComp
-Wire Wire Line
 	1100 2500 600  2500
 Wire Wire Line
-	600  2500 600  5400
+	600  2500 600  5300
 Wire Wire Line
 	1100 2600 700  2600
@@
 	1    0    0    -1
 $EndComp
-Wire Wire Line
-	1800 3800 1800 4100
 $Sheet
 S 4200 6500 1300 2300
@@
 	3200 1600 4200 1600
 Wire Wire Line
-	3000 4500 3000 6600
+	3000 4900 3000 6600
 Wire Wire Line
 	3000 6600 4100 6600
@@
 Wire Wire Line
 	9800 6900 10300 6900
-$Comp
-L Analog_Switch:ADG715 U101
-U 1 1 5AE36C1A
-P 1800 5100
-F 0 "U101" H 1150 6050 50  0000 C CNN
-F 1 "ADG715" H 2350 6050 50  0000 C CNN
-F 2 "Package_SO:TSSOP-24_4.4x7.8mm_P0.65mm" H 2800 4600 50  0001 C CIN
-F 3 "http://www.analog.com/media/en/technical-documentation/data-sheets/ADG714_715.pdf" H 1800 4900 50  0001 C CNN
-	1    1800 5100
-	1    0    0    -1
-$EndComp
-Wire Wire Line
-	1900 5900 1900 6250
-Wire Wire Line
-	800  3800 1800 3800
-Wire Wire Line
-	800  3800 800  4400
-Wire Wire Line
-	800  5300 1000 5300
+Wire Wire Line
+	800  3800 1400 3800
+Wire Wire Line
+	800  3800 800  4300
 Connection ~ 800  3800
 Wire Wire Line
-	1000 5500 700  5500
-Wire Wire Line
-	700  2600 700  5500
-Wire Wire Line
-	600  5400 1000 5400
+	700  2600 700  5400
 Wire Wire Line
 	700  5600 700  5700
@@
 	700  5700 700  6250
 Wire Wire Line
-	3000 4500 2600 4500
-Wire Wire Line
-	2600 4400 3000 4400
-Wire Wire Line
 	800  4400 1000 4400
 Connection ~ 800  4400
@@
 Connection ~ 800  4600
 Wire Wire Line
-	800  4600 800  4700
-Wire Wire Line
-	800  4700 1000 4700
-Connection ~ 800  4700
-Wire Wire Line
-	800  4700 800  4800
-Wire Wire Line
 	800  4800 1000 4800
 Connection ~ 800  4800
@@
 Wire Wire Line
 	800  5100 1000 5100
-Connection ~ 800  5100
-Wire Wire Line
-	800  5100 800  5300
-NoConn ~ 2600 4600
-NoConn ~ 2600 4700
-NoConn ~ 2600 4800
-NoConn ~ 2600 4900
-NoConn ~ 2600 5000
-NoConn ~ 2600 5100
 NoConn ~ 2500 2600
 NoConn ~ 2500 2700
@@
 Wire Wire Line
 	5500 8300 5600 8300
+$Comp
+L Power_Management:TPS22993 U101
+U 1 1 5B0BC0D7
+P 1500 5000
+F 0 "U101" H 1150 5850 50  0000 C CNN
+F 1 "TPS22993" H 1700 5850 50  0000 C CNN
+F 2 "Package_DFN_QFN:Texas_S-PWQFN-N20" H 2800 4150 50  0001 C CNN
+F 3 "http://www.ti.com/lit/gpn/tps22993" H 1400 5450 50  0001 C CNN
+	1    1500 5000
+	1    0    0    -1
+$EndComp
+Wire Wire Line
+	800  4600 800  4800
+Wire Wire Line
+	800  4300 1000 4300
+Connection ~ 800  4300
+Wire Wire Line
+	800  4300 800  4400
+Wire Wire Line
+	1400 4100 1400 3800
+Wire Wire Line
+	1500 6300 1500 5900
+Wire Wire Line
+	2000 4800 3000 4800
+Wire Wire Line
+	2000 4900 3000 4900
+Wire Wire Line
+	600  5300 1000 5300
+Wire Wire Line
+	700  5400 1000 5400
+Wire Wire Line
+	700  5600 700  5500
+Wire Wire Line
+	700  5500 1000 5500
+Connection ~ 700  5600
+Wire Wire Line
+	900  2300 900  3700
+Wire Wire Line
+	900  3700 1500 3700
+Wire Wire Line
+	1500 3700 1500 4100
+Connection ~ 900  2300
+Wire Wire Line
+	900  2300 700  2300
+$Comp
+L Venus-256-rescue:Test_Point_Flag-Connector_Specialized TP101
+U 1 1 5B1F6758
+P 2300 5300
+F 0 "TP101" H 2559 5396 50  0000 L CNN
+F 1 "VOUT3_TP" H 2559 5305 50  0000 L CNN
+F 2 "TestPoint:TestPoint_Pad_1.0x1.0mm" H 2500 5300 50  0001 C CNN
+F 3 "" H 2500 5300 50  0001 C CNN
+	1    2300 5300
+	1    0    0    -1
+$EndComp
+$Comp
+L Venus-256-rescue:Test_Point_Flag-Connector_Specialized TP102
+U 1 1 5B1F67A1
+P 2300 5500
+F 0 "TP102" H 2559 5596 50  0000 L CNN
+F 1 "VOUT4_TP" H 2559 5505 50  0000 L CNN
+F 2 "TestPoint:TestPoint_Pad_1.0x1.0mm" H 2500 5500 50  0001 C CNN
+F 3 "" H 2500 5500 50  0001 C CNN
+	1    2300 5500
+	1    0    0    -1
+$EndComp
+Wire Wire Line
+	2000 5000 2200 5000
+Wire Wire Line
+	2200 5000 2200 5300
+Wire Wire Line
+	2200 5300 2300 5300
+Wire Wire Line
+	2000 5100 2100 5100
+Wire Wire Line
+	2100 5100 2100 5500
+Wire Wire Line
+	2100 5500 2300 5500
 $EndSCHEMATC

Commit message: Updated the AD7616 symbol to match the library
Updated the AD7616 symbol to match the library
Parts:
- added JP101: VOUT1_JP, symbol Jumper:SolderJumper_2_Bridged
- added JP102: VOUT2_JP, symbol Jumper:SolderJumper_2_Bridged
Connections:
- wire segments 258 -> 262
Changed lines of the file:
@@
 $EndSheet
 $Comp
-L power:GND #PWR0106
+L power:GND #PWR0105
 U 1 1 5AE8F6FC
 P 4100 3300
-F 0 "#PWR0106" H 4100 3050 50  0001 C CNN
+F 0 "#PWR0105" H 4100 3050 50  0001 C CNN
 F 1 "GND" H 4105 3127 50  0000 C CNN
 F 2 "" H 4100 3300 50  0001 C CNN
@@
 Connection ~ 800  1000
 $Comp
-L power:GND #PWR0108
+L power:GND #PWR0107
 U 1 1 5AE90A11
 P 9900 1600
-F 0 "#PWR0108" H 9900 1350 50  0001 C CNN
+F 0 "#PWR0107" H 9900 1350 50  0001 C CNN
 F 1 "GND" H 9905 1427 50  0000 C CNN
 F 2 "" H 9900 1600 50  0001 C CNN
@@
 	9900 1400 9900 1600
 $Comp
-L power:GND #PWR0113
+L power:GND #PWR0112
 U 1 1 5AE919C7
 P 10100 1600
-F 0 "#PWR0113" H 10100 1350 50  0001 C CNN
+F 0 "#PWR0112" H 10100 1350 50  0001 C CNN
 F 1 "GND" H 10105 1427 50  0000 C CNN
 F 2 "" H 10100 1600 50  0001 C CNN
@@
 	10400 2300 9800 2300
 $Comp
-L power:GND #PWR0109
+L power:GND #PWR0108
 U 1 1 5AE958F1
 P 9900 2900
-F 0 "#PWR0109" H 9900 2650 50  0001 C CNN
+F 0 "#PWR0108" H 9900 2650 50  0001 C CNN
 F 1 "GND" H 9905 2727 50  0000 C CNN
 F 2 "" H 9900 2900 50  0001 C CNN
@@
 	9900 2700 9900 2900
 $Comp
-L power:GND #PWR0114
+L power:GND #PWR0113
 U 1 1 5AE958F9
 P 10100 2900
-F 0 "#PWR0114" H 10100 2650 50  0001 C CNN
+F 0 "#PWR0113" H 10100 2650 50  0001 C CNN
 F 1 "GND" H 10105 2727 50  0000 C CNN
 F 2 "" H 10100 2900 50  0001 C CNN
@@
 	10400 3600 9800 3600
 $Comp
-L power:GND #PWR0110
+L power:GND #PWR0109
 U 1 1 5AE96319
 P 9900 4200
-F 0 "#PWR0110" H 9900 3950 50  0001 C CNN
+F 0 "#PWR0109" H 9900 3950 50  0001 C CNN
 F 1 "GND" H 9905 4027 50  0000 C CNN
 F 2 "" H 9900 4200 50  0001 C CNN
@@
 	9900 4000 9900 4200
 $Comp
-L power:GND #PWR0115
+L power:GND #PWR0114
 U 1 1 5AE96321
 P 10100 4200
-F 0 "#PWR0115" H 10100 3950 50  0001 C CNN
+F 0 "#PWR0114" H 10100 3950 50  0001 C CNN
 F 1 "GND" H 10105 4027 50  0000 C CNN
 F 2 "" H 10100 4200 50  0001 C CNN
@@
 	10400 4900 9800 4900
 $Comp
-L power:GND #PWR0111
+L power:GND #PWR0110
 U 1 1 5AE96EDB
 P 9900 5500
-F 0 "#PWR0111" H 9900 5250 50  0001 C CNN
+F 0 "#PWR0110" H 9900 5250 50  0001 C CNN
 F 1 "GND" H 9905 5327 50  0000 C CNN
 F 2 "" H 9900 5500 50  0001 C CNN
@@
 	9900 5300 9900 5500
 $Comp
-L power:GND #PWR0116
+L power:GND #PWR0115
 U 1 1 5AE96EE3
 P 10100 5500
-F 0 "#PWR0116" H 10100 5250 50  0001 C CNN
+F 0 "#PWR0115" H 10100 5250 50  0001 C CNN
 F 1 "GND" H 10105 5327 50  0000 C CNN
 F 2 "" H 10100 5500 50  0001 C CNN
@@
 	4100 1100 4100 1000
 Wire Wire Line
-	3000 1000 3000 4800
+	3000 1000 3000 4500
 Wire Wire Line
 	3000 1000 4100 1000
@@
 $EndSheet
 $Comp
-L power:GND #PWR0107
+L power:GND #PWR0106
 U 1 1 5AF03082
 P 4100 8950
-F 0 "#PWR0107" H 4100 8700 50  0001 C CNN
+F 0 "#PWR0106" H 4100 8700 50  0001 C CNN
 F 1 "GND" H 4105 8777 50  0000 C CNN
 F 2 "" H 4100 8950 50  0001 C CNN
@@
 	8000 7500 8500 7500
 $Comp
-L power:GND #PWR0112
+L power:GND #PWR0111
 U 1 1 5B09A94C
 P 9900 7250
-F 0 "#PWR0112" H 9900 7000 50  0001 C CNN
+F 0 "#PWR0111" H 9900 7000 50  0001 C CNN
 F 1 "GND" H 9905 7077 50  0000 C CNN
 F 2 "" H 9900 7250 50  0001 C CNN
@@
 	9900 7000 9900 7250
 $Comp
-L power:GND #PWR0117
+L power:GND #PWR0116
 U 1 1 5B09A954
 P 10100 7250
-F 0 "#PWR0117" H 10100 7000 50  0001 C CNN
+F 0 "#PWR0116" H 10100 7000 50  0001 C CNN
 F 1 "GND" H 10105 7077 50  0000 C CNN
 F 2 "" H 10100 7250 50  0001 C CNN
@@
 	1500 6300 1500 5900
 Wire Wire Line
-	2000 4800 3000 4800
-Wire Wire Line
-	2000 4900 3000 4900
-Wire Wire Line
 	600  5300 1000 5300
 Wire Wire Line
@@
 Wire Wire Line
 	2100 5500 2300 5500
+$Comp
+L Jumper:SolderJumper_2_Bridged JP101
+U 1 1 5B23A184
+P 2450 4500
+F 0 "JP101" H 2600 4550 50  0000 C CNN
+F 1 "VOUT1_JP" H 2700 4400 50  0000 C CNN
+F 2 "" H 2450 4500 50  0001 C CNN
+F 3 "~" H 2450 4500 50  0001 C CNN
+	1    2450 4500
+	1    0    0    -1
+$EndComp
+$Comp
+L Jumper:SolderJumper_2_Bridged JP102
+U 1 1 5B23A20E
+P 2450 4900
+F 0 "JP102" H 2600 4950 50  0000 C CNN
+F 1 "VOUT2_JP" H 2700 4800 50  0000 C CNN
+F 2 "" H 2450 4900 50  0001 C CNN
+F 3 "~" H 2450 4900 50  0001 C CNN
+	1    2450 4900
+	1    0    0    -1
+$EndComp
+Wire Wire Line
+	2000 4900 2300 4900
+Wire Wire Line
+	2600 4900 3000 4900
+Wire Wire Line
+	2000 4800 2200 4800
+Wire Wire Line
+	2200 4800 2200 4500
+Wire Wire Line
+	2200 4500 2300 4500
+Wire Wire Line
+	3000 4500 2600 4500
 $EndSCHEMATC

Commit message: Added jumpers to TPS22993
Parts:
- JP101, JP102: footprint (none) -> Jumper:SolderJumper-2_P1.3mm_Bridged2Bar_Pad1.0x1.5mm
Changed lines of the file:
@@
 F 0 "JP101" H 2600 4550 50  0000 C CNN
 F 1 "VOUT1_JP" H 2700 4400 50  0000 C CNN
-F 2 "" H 2450 4500 50  0001 C CNN
+F 2 "Jumper:SolderJumper-2_P1.3mm_Bridged2Bar_Pad1.0x1.5mm" H 2450 4500 50  0001 C CNN
 F 3 "~" H 2450 4500 50  0001 C CNN
 	1    2450 4500
@@
 F 0 "JP102" H 2600 4950 50  0000 C CNN
 F 1 "VOUT2_JP" H 2700 4800 50  0000 C CNN
-F 2 "" H 2450 4900 50  0001 C CNN
+F 2 "Jumper:SolderJumper-2_P1.3mm_Bridged2Bar_Pad1.0x1.5mm" H 2450 4900 50  0001 C CNN
 F 3 "~" H 2450 4900 50  0001 C CNN
 	1    2450 4900
