File: Hardware/Schematics/BBDProto06/Venus-256/CellSlave.sch (KiCad schematic (older format))
At the start: 3 parts, among them J100 CH00, J101 CH01

Commit message: Updated the Cell Master and Slave schematics
Updated the Cell Master and Slave schematics
Parts:
- removed J100: CH00, symbol Connector_Generic:Conn_01x01
- removed J101: CH01, symbol Connector_Generic:Conn_01x01
- added C?: 10uF,X5R, symbol Device:C_Small
- added C? (x2): 10uF, symbol Device:C_Small
- added C?: 0.1uF,X8R, symbol Device:C_Small
- added J?: S01, symbol Connector_Generic:Conn_01x01
- added J?: S02, symbol Connector_Generic:Conn_01x01
- added J?: S03, symbol Connector_Generic:Conn_01x01
- added J?: S04, symbol Connector_Generic:Conn_01x01
- added J?: S05, symbol Connector_Generic:Conn_01x01
- added J?: S06, symbol Connector_Generic:Conn_01x01
- added J?: S07, symbol Connector_Generic:Conn_01x01
- added J?: S08, symbol Connector_Generic:Conn_01x01
- added J?: S09, symbol Connector_Generic:Conn_01x01
- added J?: S10, symbol Connector_Generic:Conn_01x01
- added J?: S11, symbol Connector_Generic:Conn_01x01
- added J?: S12, symbol Connector_Generic:Conn_01x01
- added J?: S13, symbol Connector_Generic:Conn_01x01
- added J?: S14, symbol Connector_Generic:Conn_01x01
- added J?: S15, symbol Connector_Generic:Conn_01x01
- added J?: S16, symbol Connector_Generic:Conn_01x01
Connections:
- net labels added: ADC_REF_OUT, AGND, BUSY, CONVST, DGND, SCLK, SDI, SDOA, SGND, VCC_5V0, VDRIVE_3V3, ~CS, ~RESET
- wire segments 0 -> 125
- no-connect marks 0 -> 1

Commit message: Added Cell Slave capacitors
Added Cell Slave capacitors
Parts:
- added C? (x6): 0.1uF, symbol Device:C_Small
- added C? (x6): 10uF, symbol Device:C_Small
- C?: value 10uF -> 0.1uF
Connections:
- wire segments 125 -> 193

Commit message: Completed the Cell Master and Slave schematics
Completed the Cell Master and Slave schematics
Parts:
- added J?: ADC_REF_OUT, symbol Connector_Generic:Conn_01x01
Connections:
- net labels removed: ADC_REF_OUT
Changed lines of the file:
@@
 $Descr A4 11693 8268
 encoding utf-8
-Sheet 5 5
+Sheet 4 8
 Title "Cell Slave"
 Date "2018-04-26"
@@
 Text HLabel 4700 2500 2    50   Input ~ 0
 VDRIVE_3V3
-Text HLabel 5900 2000 2    50   Output ~ 0
-ADC_REF_OUT
 Text HLabel 5000 2100 2    50   UnSpc ~ 0
 AGND
@@
 Wire Wire Line
 	2800 1600 2800 1700
+$Comp
+L Connector_Generic:Conn_01x01 J?
+U 1 1 5AE85F26
+P 6100 2000
+F 0 "J?" H 6179 2042 50  0000 L CNN
+F 1 "ADC_REF_OUT" H 6179 1951 50  0000 L CNN
+F 2 "" H 6100 2000 50  0001 C CNN
+F 3 "~" H 6100 2000 50  0001 C CNN
+	1    6100 2000
+	1    0    0    -1
+$EndComp
 $EndSCHEMATC

Commit message: Started to rearrange the Venus-256 PCB
Started to rearrange the Venus-256 PCB
Parts:
- removed J?: ADC_REF_OUT, symbol Connector_Generic:Conn_01x01
- added TP1: ADC_REF_OUT, TestPoint:TestPoint_Pad_1.5x1.5mm, symbol Connector_Specialized:Test_Point
- C1, C10, C11, C12, C13, C14, C15, C16, C2, C3, C4, C5, C6, C7, C8, C9: renamed from C?; footprint (none) -> Capacitor_SMD:C_0603_1608Metric_Pad0.84x1.00mm_HandSolder
- J10, J11, J12, J13, J14, J15, J16, J17, J18, J3, J4, J5, J6, J7, J8, J9: renamed from J?; footprint (none) -> Connector_Wire:SolderWirePad_single_0-8mmDrill
- gave numbers to parts that had none: 1

Commit message: Added a 5th cell-slave
Added a 5th cell-slave
Parts:
- removed J10: S08, Connector_Wire:SolderWirePad_single_0-8mmDrill, symbol Connector_Generic:Conn_01x01
- removed J11: S09, Connector_Wire:SolderWirePad_single_0-8mmDrill, symbol Connector_Generic:Conn_01x01
- removed J12: S10, Connector_Wire:SolderWirePad_single_0-8mmDrill, symbol Connector_Generic:Conn_01x01
- removed J13: S11, Connector_Wire:SolderWirePad_single_0-8mmDrill, symbol Connector_Generic:Conn_01x01
- removed J14: S12, Connector_Wire:SolderWirePad_single_0-8mmDrill, symbol Connector_Generic:Conn_01x01
- removed J15: S13, Connector_Wire:SolderWirePad_single_0-8mmDrill, symbol Connector_Generic:Conn_01x01
- removed J16: S14, Connector_Wire:SolderWirePad_single_0-8mmDrill, symbol Connector_Generic:Conn_01x01
- removed J17: S15, Connector_Wire:SolderWirePad_single_0-8mmDrill, symbol Connector_Generic:Conn_01x01
- removed J18: S16, Connector_Wire:SolderWirePad_single_0-8mmDrill, symbol Connector_Generic:Conn_01x01
- removed J3: S01, Connector_Wire:SolderWirePad_single_0-8mmDrill, symbol Connector_Generic:Conn_01x01
- removed J4: S02, Connector_Wire:SolderWirePad_single_0-8mmDrill, symbol Connector_Generic:Conn_01x01
- removed J5: S03, Connector_Wire:SolderWirePad_single_0-8mmDrill, symbol Connector_Generic:Conn_01x01
- removed J6: S04, Connector_Wire:SolderWirePad_single_0-8mmDrill, symbol Connector_Generic:Conn_01x01
- removed J7: S05, Connector_Wire:SolderWirePad_single_0-8mmDrill, symbol Connector_Generic:Conn_01x01
- removed J8: S06, Connector_Wire:SolderWirePad_single_0-8mmDrill, symbol Connector_Generic:Conn_01x01
- removed J9: S07, Connector_Wire:SolderWirePad_single_0-8mmDrill, symbol Connector_Generic:Conn_01x01
- added TP1001: S01, TestPoint:TestPoint_Pad_1.5x1.5mm, symbol Connector_Specialized:Test_Point_Flag
- added TP1002: S02, TestPoint:TestPoint_Pad_1.5x1.5mm, symbol Connector_Specialized:Test_Point_Flag
- added TP1003: S03, TestPoint:TestPoint_Pad_1.5x1.5mm, symbol Connector_Specialized:Test_Point_Flag
- added TP1004: S04, TestPoint:TestPoint_Pad_1.5x1.5mm, symbol Connector_Specialized:Test_Point_Flag
- added TP1005: S05, TestPoint:TestPoint_Pad_1.5x1.5mm, symbol Connector_Specialized:Test_Point_Flag
- added TP1006: S06, TestPoint:TestPoint_Pad_1.5x1.5mm, symbol Connector_Specialized:Test_Point_Flag
- added TP1007: S07, TestPoint:TestPoint_Pad_1.5x1.5mm, symbol Connector_Specialized:Test_Point_Flag
- added TP1008: S08, TestPoint:TestPoint_Pad_1.5x1.5mm, symbol Connector_Specialized:Test_Point_Flag
- added TP1009: S09, TestPoint:TestPoint_Pad_1.5x1.5mm, symbol Connector_Specialized:Test_Point_Flag
- added TP1010: S10, TestPoint:TestPoint_Pad_1.5x1.5mm, symbol Connector_Specialized:Test_Point_Flag
- added TP1011: S11, TestPoint:TestPoint_Pad_1.5x1.5mm, symbol Connector_Specialized:Test_Point_Flag
- added TP1012: S12, TestPoint:TestPoint_Pad_1.5x1.5mm, symbol Connector_Specialized:Test_Point_Flag
- added TP1013: S13, TestPoint:TestPoint_Pad_1.5x1.5mm, symbol Connector_Specialized:Test_Point_Flag
- added TP1014: S14, TestPoint:TestPoint_Pad_1.5x1.5mm, symbol Connector_Specialized:Test_Point_Flag
- added TP1015: S15, TestPoint:TestPoint_Pad_1.5x1.5mm, symbol Connector_Specialized:Test_Point_Flag
- added TP1016: S16, TestPoint:TestPoint_Pad_1.5x1.5mm, symbol Connector_Specialized:Test_Point_Flag
- renumbered C1 to C1001, C2 to C1002, C3 to C1003, C4 to C1004, C5 to C1005, C6 to C1006, C7 to C1007, C8 to C1008, C9 to C1009, C10 to C1010, C11 to C1011, C12 to C1012, C13 to C1013, C14 to C1014, C15 to C1015, C16 to C1016, TP1 to TP1017, U2 to U1001

Commit message: Updated the AD7616 and its Cell Slave schematics
Updated the AD7616 and its Cell Slave schematics
Parts:
- TP701: renamed from TP1001; symbol Connector_Specialized:Test_Point_Flag -> Venus-256-rescue:Test_Point_Flag-Connector_Specialized
- TP702: renamed from TP1002; symbol Connector_Specialized:Test_Point_Flag -> Venus-256-rescue:Test_Point_Flag-Connector_Specialized
- TP703: renamed from TP1003; symbol Connector_Specialized:Test_Point_Flag -> Venus-256-rescue:Test_Point_Flag-Connector_Specialized
- TP704: renamed from TP1004; symbol Connector_Specialized:Test_Point_Flag -> Venus-256-rescue:Test_Point_Flag-Connector_Specialized
- TP705: renamed from TP1005; symbol Connector_Specialized:Test_Point_Flag -> Venus-256-rescue:Test_Point_Flag-Connector_Specialized
- TP706: renamed from TP1006; symbol Connector_Specialized:Test_Point_Flag -> Venus-256-rescue:Test_Point_Flag-Connector_Specialized
- TP707: renamed from TP1007; symbol Connector_Specialized:Test_Point_Flag -> Venus-256-rescue:Test_Point_Flag-Connector_Specialized
- TP708: renamed from TP1008; symbol Connector_Specialized:Test_Point_Flag -> Venus-256-rescue:Test_Point_Flag-Connector_Specialized
- TP709: renamed from TP1009; symbol Connector_Specialized:Test_Point_Flag -> Venus-256-rescue:Test_Point_Flag-Connector_Specialized
- TP710: renamed from TP1010; symbol Connector_Specialized:Test_Point_Flag -> Venus-256-rescue:Test_Point_Flag-Connector_Specialized
- TP711: renamed from TP1011; symbol Connector_Specialized:Test_Point_Flag -> Venus-256-rescue:Test_Point_Flag-Connector_Specialized
- TP712: renamed from TP1012; symbol Connector_Specialized:Test_Point_Flag -> Venus-256-rescue:Test_Point_Flag-Connector_Specialized
- TP713: renamed from TP1013; symbol Connector_Specialized:Test_Point_Flag -> Venus-256-rescue:Test_Point_Flag-Connector_Specialized
- TP714: renamed from TP1014; symbol Connector_Specialized:Test_Point_Flag -> Venus-256-rescue:Test_Point_Flag-Connector_Specialized
- TP715: renamed from TP1015; symbol Connector_Specialized:Test_Point_Flag -> Venus-256-rescue:Test_Point_Flag-Connector_Specialized
- TP716: renamed from TP1016; symbol Connector_Specialized:Test_Point_Flag -> Venus-256-rescue:Test_Point_Flag-Connector_Specialized
- TP717: renamed from TP1017; symbol Connector_Specialized:Test_Point -> Venus-256-rescue:Test_Point-Connector_Specialized
- renumbered C1001 to C701, C1002 to C702, C1003 to C703, C1004 to C704, C1007 to C705, C1008 to C706, C1009 to C707, C1010 to C708, C1006 to C709, C1005 to C710, C1014 to C711, C1011 to C712, C1012 to C713, C1015 to C714, C1013 to C715, C1016 to C716, U1001 to U701
Connections:
- wire segments 193 -> 142

Commit message: Moved the capacitors around
Parts:
- TP701, TP702, TP703, TP704, TP705, TP706, TP707, TP708, TP709, TP710, TP711, TP712, TP713, TP714, TP715, TP716, TP717: footprint TestPoint:TestPoint_Pad_1.5x1.5mm -> TestPoint:TestPoint_Pad_1.0x1.0mm
