File: Hardware/Schematics/BBDProto06/Venus-256/CellSlave.sch (KiCad schematic (older format))
At the start: 34 parts, among them U701 AD7616

Commit message: Updated the AD7616 symbol to match the library
Updated the AD7616 symbol to match the library
Parts:
- renumbered C715 to C401, C713 to C402, C711 to C403, C712 to C404, C701 to C405, C702 to C406, C703 to C407, C704 to C408, C705 to C409, C706 to C410, C707 to C411, C708 to C412, C709 to C413, C710 to C414, C714 to C415, C716 to C416, TP717 to TP401, TP701 to TP402, TP702 to TP403, TP703 to TP404, TP704 to TP405, TP705 to TP406, TP706 to TP407, TP707 to TP408, TP708 to TP409, TP709 to TP410, TP710 to TP411, TP711 to TP412, TP712 to TP413, TP713 to TP414, TP714 to TP415, TP715 to TP416, TP716 to TP417, U701 to U401
Other:
- moved on the sheet: TP1001, TP1002, TP1003, TP1004, TP1005, TP1006, TP1007, TP1008, TP1009, TP1010, TP1011, TP1012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

Commit message: Added the big pads behind the sensors
Parts:
- renumbered TP402 to TP401, TP403 to TP402, TP404 to TP403, TP405 to TP404, TP406 to TP405, TP407 to TP406, TP408 to TP407, TP409 to TP408, TP410 to TP409, TP411 to TP410, TP412 to TP411, TP413 to TP412, TP414 to TP413, TP415 to TP414, TP416 to TP415, TP417 to TP416, TP401 to TP417
Other:
- moved on the sheet: TP401, TP402, TP403, TP404, TP405, TP406, TP407, TP408, TP409, TP410, TP411, TP412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

Commit message: Switched around the ADC channels to make the PCB simpler
Other:
- moved on the sheet: TP401, TP402, TP403, TP404, TP405, TP406, TP407, TP408, TP409, TP410, TP411, TP412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
