File: Hardware/Schematics/BBDProto06/Venus-256/RaspberryPiGPIOHeader.sch (KiCad schematic (older format))
At the start: 1 part

Commit message: Updated the Cell Master and Slave schematics
Updated the Cell Master and Slave schematics
Connections:
- net labels added: DC_POWER_5V0
- wire segments 17 -> 19
Changed lines of the file:
@@
 $Descr A4 11693 8268
 encoding utf-8
-Sheet 3 3
+Sheet 3 5
 Title "Raspberry Pi GOIP Header"
 Date "2018-04-27"
@@
 Wire Wire Line
 	2400 1300 2700 1300
+Text HLabel 2700 1100 2    50   Output ~ 0
+DC_POWER_5V0
+Text HLabel 2700 1200 2    50   Output ~ 0
+DC_POWER_5V0
+Wire Wire Line
+	2400 1100 2700 1100
+Wire Wire Line
+	2400 1200 2700 1200
 $EndSCHEMATC

Commit message: Started to rearrange the Venus-256 PCB
Started to rearrange the Venus-256 PCB
Parts:
- J1: renamed from J?; footprint (none) -> Connector_PinHeader_2.54mm:PinHeader_2x20_P2.54mm_Vertical
Changed lines of the file:
@@
 $Descr A4 11693 8268
 encoding utf-8
-Sheet 3 8
+Sheet 3 9
 Title "Raspberry Pi GOIP Header"
 Date "2018-04-27"
@@
 $EndDescr
 $Comp
-L Connector_Generic:Conn_02x20_Odd_Even J?
+L Connector_Generic:Conn_02x20_Odd_Even J1
 U 1 1 5AE76166
 P 2100 2000
-F 0 "J?" H 2150 3000 50  0000 C CNN
+F 0 "J1" H 2150 3000 50  0000 C CNN
 F 1 "RaspberryPi header" H 2150 900 50  0000 C CNN
-F 2 "" H 2100 2000 50  0001 C CNN
+F 2 "Connector_PinHeader_2.54mm:PinHeader_2x20_P2.54mm_Vertical" H 2100 2000 50  0001 C CNN
 F 3 "~" H 2100 2000 50  0001 C CNN
 	1    2100 2000

Commit message: Updated the AD7616 and its Cell Slave schematics
Updated the AD7616 and its Cell Slave schematics
Parts:
- J201: renamed from J1; footprint Connector_PinHeader_2.54mm:PinHeader_2x20_P2.54mm_Vertical -> Connector_PinHeader_2.54mm:PinHeader_2x20_P2.54mm_Horizontal
Changed lines of the file:
@@
 $EndDescr
 $Comp
-L Connector_Generic:Conn_02x20_Odd_Even J1
+L Connector_Generic:Conn_02x20_Odd_Even J201
 U 1 1 5AE76166
 P 2100 2000
-F 0 "J1" H 2150 3000 50  0000 C CNN
+F 0 "J201" H 2150 3000 50  0000 C CNN
 F 1 "RaspberryPi header" H 2150 900 50  0000 C CNN
-F 2 "Connector_PinHeader_2.54mm:PinHeader_2x20_P2.54mm_Vertical" H 2100 2000 50  0001 C CNN
+F 2 "Connector_PinHeader_2.54mm:PinHeader_2x20_P2.54mm_Horizontal" H 2100 2000 50  0001 C CNN
 F 3 "~" H 2100 2000 50  0001 C CNN
 	1    2100 2000

Commit message: Fixed many rules check errors and changed the footprint of test points
Connections:
- no-connect marks 0 -> 21
Changed lines of the file:
@@
 Wire Wire Line
 	2400 1200 2700 1200
+NoConn ~ 1900 1400
+NoConn ~ 1900 1600
+NoConn ~ 1900 1700
+NoConn ~ 1900 1800
+NoConn ~ 2400 1400
+NoConn ~ 2400 1500
+NoConn ~ 2400 1600
+NoConn ~ 2400 1800
+NoConn ~ 2400 1900
+NoConn ~ 2400 2100
+NoConn ~ 2400 2200
+NoConn ~ 2400 2300
+NoConn ~ 2400 2600
+NoConn ~ 2400 2800
+NoConn ~ 2400 2900
+NoConn ~ 2400 3000
+NoConn ~ 1900 2900
+NoConn ~ 1900 2800
+NoConn ~ 1900 2700
+NoConn ~ 1900 2600
+NoConn ~ 1900 2500
 $EndSCHEMATC
