File: Hardware/Schematics/BBDProto06/Venus-256/CellMaster.sch (KiCad schematic (older format))
At the start: 21 parts, among them U1 ATSAME70Q21A-AN

Commit message: Completed the Cell Master and Slave schematics
Completed the Cell Master and Slave schematics
Parts:
- added J?: AFE0_AD0, symbol Connector_Generic:Conn_01x01
- added J?: AFE0_AD1, symbol Connector_Generic:Conn_01x01
Connections:
- net labels added: ADC_BUSY0, ADC_BUSY1, ADC_BUSY2, ADC_BUSY3, ADC_CONVST0, ADC_CONVST1, ADC_CONVST2, ADC_CONVST3, ADC_RESET
- net labels removed: AFE0_AD0, AFE0_AD1, DAC1, USBD+, USBD-
- wire segments 155 -> 161
Changed lines of the file:
@@
 $Descr A3 16535 11693
 encoding utf-8
-Sheet 2 5
+Sheet 5 8
 Title "Venus-256 / Cell Master"
 Date "2018-04-06"
@@
 Wire Wire Line
 	5700 7600 6000 7600
-Text HLabel 5700 8900 0    50   Output ~ 0
-USBD+
-Text HLabel 5700 9000 0    50   Output ~ 0
-USBD-
-Wire Wire Line
-	5700 8900 6000 8900
-Wire Wire Line
-	5700 9000 6000 9000
 Text HLabel 5700 9300 0    50   Input ~ 0
 TARGET_RESET
@@
 Text HLabel 8900 6000 2    50   Output ~ 0
 SPI1_SPCK
-Text HLabel 5700 5700 0    50   Input ~ 0
-AFE0_AD1
-Text HLabel 8900 9900 2    50   Input ~ 0
-AFE0_AD0
-Text HLabel 8900 6900 2    50   Output ~ 0
-DAC1
 Wire Wire Line
 	5700 5700 6000 5700
@@
 Wire Wire Line
 	8600 6600 8900 6600
-Wire Wire Line
-	8600 6900 8900 6900
 Wire Wire Line
 	6000 7000 5000 7000
@@
 	4800 8000 5000 8000
 Connection ~ 5000 8000
+$Comp
+L Connector_Generic:Conn_01x01 J?
+U 1 1 5AE3AAE9
+P 9100 9900
+F 0 "J?" H 9180 9942 50  0000 L CNN
+F 1 "AFE0_AD0" H 9180 9851 50  0000 L CNN
+F 2 "" H 9100 9900 50  0001 C CNN
+F 3 "~" H 9100 9900 50  0001 C CNN
+	1    9100 9900
+	1    0    0    -1
+$EndComp
+$Comp
+L Connector_Generic:Conn_01x01 J?
+U 1 1 5AE3AD89
+P 5500 5700
+F 0 "J?" H 5420 5475 50  0000 C CNN
+F 1 "AFE0_AD1" H 5420 5566 50  0000 C CNN
+F 2 "" H 5500 5700 50  0001 C CNN
+F 3 "~" H 5500 5700 50  0001 C CNN
+	1    5500 5700
+	-1   0    0    1
+$EndComp
+Text HLabel 5700 8200 0    50   Output ~ 0
+ADC_CONVST0
+Wire Wire Line
+	5700 8200 6000 8200
+Text HLabel 5700 5900 0    50   Input ~ 0
+ADC_BUSY0
+Text HLabel 5700 6000 0    50   Input ~ 0
+ADC_BUSY1
+Text HLabel 5700 6100 0    50   Input ~ 0
+ADC_BUSY2
+Text HLabel 5700 6200 0    50   Input ~ 0
+ADC_BUSY3
+Wire Wire Line
+	5700 5900 6000 5900
+Wire Wire Line
+	5700 6000 6000 6000
+Wire Wire Line
+	5700 6100 6000 6100
+Wire Wire Line
+	5700 6200 6000 6200
+Text HLabel 5700 8300 0    50   Output ~ 0
+ADC_CONVST1
+Text HLabel 5700 8400 0    50   Output ~ 0
+ADC_CONVST2
+Text HLabel 5700 8500 0    50   Output ~ 0
+ADC_CONVST3
+Wire Wire Line
+	5700 8300 6000 8300
+Wire Wire Line
+	5700 8400 6000 8400
+Wire Wire Line
+	5700 8500 6000 8500
+Text HLabel 5700 6300 0    50   Input ~ 0
+ADC_RESET
+Wire Wire Line
+	5700 6300 6000 6300
 $EndSCHEMATC

Commit message: Started to rearrange the Venus-256 PCB
Started to rearrange the Venus-256 PCB
Parts:
- removed J?: AFE0_AD0, symbol Connector_Generic:Conn_01x01
- removed J?: AFE0_AD1, symbol Connector_Generic:Conn_01x01
- removed J?: ADVREF, symbol Connector_Generic:Conn_01x01
- added TP2: ADVREF, TestPoint:TestPoint_Pad_1.5x1.5mm, symbol Connector_Specialized:Test_Point
- added TP3: AFE0_AD1, TestPoint:TestPoint_Pad_1.5x1.5mm, symbol Connector_Specialized:Test_Point
- added TP4: AFE0_AD0, TestPoint:TestPoint_Pad_1.5x1.5mm, symbol Connector_Specialized:Test_Point
- C17, C18, C19, C20, C21, C22, C23, C24, C25, C26, C27, C28, C29, C30, C31, C32: renamed from C?; footprint (none) -> Capacitor_SMD:C_0603_1608Metric_Pad0.84x1.00mm_HandSolder
- D1: renamed from D?; footprint (none) -> LED_SMD:LED_RGB_1210
- L1: renamed from L200; footprint (none) -> Inductor_SMD:L_0603_1608Metric_Pad0.84x1.00mm_HandSolder
- R5: renamed from R?; footprint (none) -> Resistor_SMD:R_0603_1608Metric_Pad0.84x1.00mm_HandSolder
- renumbered U1 to U3

Commit message: Added a 5th cell-slave
Added a 5th cell-slave
Parts:
- renumbered C17 to C501, C18 to C502, C19 to C503, C20 to C504, C21 to C505, C22 to C506, C23 to C507, C24 to C508, C25 to C509, C26 to C510, C27 to C511, C28 to C512, C29 to C513, C30 to C514, C31 to C515, C32 to C516, D1 to D501, L1 to L501, R5 to R501, TP4 to TP501, TP3 to TP502, TP2 to TP503, U3 to U501
Connections:
- wire segments 161 -> 168

Commit message: Updated the AD7616 and its Cell Slave schematics
Updated the AD7616 and its Cell Slave schematics
Parts:
- TP501, TP502, TP503: symbol Connector_Specialized:Test_Point -> Venus-256-rescue:Test_Point-Connector_Specialized
- U501: symbol MCU_Microchip_SAME:ATSAME70Q21A-AN -> Venus-256-rescue:ATSAME70Q21A-AN-MCU_Microchip_SAME
Changed lines of the file:
@@
 $Descr A3 16535 11693
 encoding utf-8
-Sheet 9 10
+Sheet 5 10
 Title "Venus-256: Cell Master"
 Date "2018-05-02"
@@
 	7300 900  7000 900
 $Comp
-L MCU_Microchip_SAME:ATSAME70Q21A-AN U501
+L Venus-256-rescue:ATSAME70Q21A-AN-MCU_Microchip_SAME U501
 U 1 1 5ACBEA02
 P 7300 6800
@@
 	5700 6300 6000 6300
 $Comp
-L Connector_Specialized:Test_Point TP502
+L Venus-256-rescue:Test_Point-Connector_Specialized TP502
 U 1 1 5AE7EA0D
 P 3100 9700
@@
 $EndComp
 $Comp
-L Connector_Specialized:Test_Point TP501
+L Venus-256-rescue:Test_Point-Connector_Specialized TP501
 U 1 1 5AE7EBD0
 P 3100 9300
@@
 $EndComp
 $Comp
-L Connector_Specialized:Test_Point TP503
+L Venus-256-rescue:Test_Point-Connector_Specialized TP503
 U 1 1 5AE7F482
 P 3100 10100

Commit message: Moved the capacitors around
Parts:
- TP501, TP502, TP503: footprint TestPoint:TestPoint_Pad_1.5x1.5mm -> TestPoint:TestPoint_Pad_1.0x1.0mm
Changed lines of the file:
@@
 AR Path="/5AE473C8/5AE1DB3B" Ref="C514"  Part="1"
 AR Path="/5AF0307C/5AE1DB3B" Ref="C914"  Part="1"
-F 0 "C914" H 7100 2200 50  0000 L CNN
+F 0 "C514" H 7100 2200 50  0000 L CNN
 F 1 "100nF" H 7100 2000 50  0000 L CNN
 F 2 "Capacitor_SMD:C_0603_1608Metric_Pad0.84x1.00mm_HandSolder" H 7100 2100 50  0001 C CNN
@@
 AR Path="/5AE473C8/5AE23144" Ref="C512"  Part="1"
 AR Path="/5AF0307C/5AE23144" Ref="C912"  Part="1"
-F 0 "C912" H 6800 2200 50  0000 L CNN
+F 0 "C512" H 6800 2200 50  0000 L CNN
 F 1 "100nF" H 6800 2000 50  0000 L CNN
 F 2 "Capacitor_SMD:C_0603_1608Metric_Pad0.84x1.00mm_HandSolder" H 6800 2100 50  0001 C CNN
@@
 AR Path="/5AE473C8/5AE23174" Ref="C510"  Part="1"
 AR Path="/5AF0307C/5AE23174" Ref="C910"  Part="1"
-F 0 "C910" H 6500 2200 50  0000 L CNN
+F 0 "C510" H 6500 2200 50  0000 L CNN
 F 1 "100nF" H 6500 2000 50  0000 L CNN
 F 2 "Capacitor_SMD:C_0603_1608Metric_Pad0.84x1.00mm_HandSolder" H 6500 2100 50  0001 C CNN
@@
 AR Path="/5AE473C8/5AE231A2" Ref="C508"  Part="1"
 AR Path="/5AF0307C/5AE231A2" Ref="C908"  Part="1"
-F 0 "C908" H 6200 2200 50  0000 L CNN
+F 0 "C508" H 6200 2200 50  0000 L CNN
 F 1 "100nF" H 6200 2000 50  0000 L CNN
 F 2 "Capacitor_SMD:C_0603_1608Metric_Pad0.84x1.00mm_HandSolder" H 6200 2100 50  0001 C CNN
@@
 AR Path="/5AE473C8/5AE231D6" Ref="C507"  Part="1"
 AR Path="/5AF0307C/5AE231D6" Ref="C907"  Part="1"
-F 0 "C907" H 5900 2200 50  0000 L CNN
+F 0 "C507" H 5900 2200 50  0000 L CNN
 F 1 "100nF" H 5900 2000 50  0000 L CNN
 F 2 "Capacitor_SMD:C_0603_1608Metric_Pad0.84x1.00mm_HandSolder" H 5900 2100 50  0001 C CNN
@@
 AR Path="/5AE473C8/5AE23204" Ref="C506"  Part="1"
 AR Path="/5AF0307C/5AE23204" Ref="C906"  Part="1"
-F 0 "C906" H 5600 2200 50  0000 L CNN
+F 0 "C506" H 5600 2200 50  0000 L CNN
 F 1 "100nF" H 5600 2000 50  0000 L CNN
 F 2 "Capacitor_SMD:C_0603_1608Metric_Pad0.84x1.00mm_HandSolder" H 5600 2100 50  0001 C CNN
@@
 AR Path="/5AE473C8/5AE23234" Ref="C504"  Part="1"
 AR Path="/5AF0307C/5AE23234" Ref="C904"  Part="1"
-F 0 "C904" H 5300 2200 50  0000 L CNN
+F 0 "C504" H 5300 2200 50  0000 L CNN
 F 1 "100nF" H 5300 2000 50  0000 L CNN
 F 2 "Capacitor_SMD:C_0603_1608Metric_Pad0.84x1.00mm_HandSolder" H 5300 2100 50  0001 C CNN
@@
 AR Path="/5AE473C8/5AE23266" Ref="C503"  Part="1"
 AR Path="/5AF0307C/5AE23266" Ref="C903"  Part="1"
-F 0 "C903" H 5000 2200 50  0000 L CNN
+F 0 "C503" H 5000 2200 50  0000 L CNN
 F 1 "100nF" H 5000 2000 50  0000 L CNN
 F 2 "Capacitor_SMD:C_0603_1608Metric_Pad0.84x1.00mm_HandSolder" H 5000 2100 50  0001 C CNN
@@
 AR Path="/5AE473C8/5AE2329A" Ref="C501"  Part="1"
 AR Path="/5AF0307C/5AE2329A" Ref="C901"  Part="1"
-F 0 "C901" H 4700 2200 50  0000 L CNN
+F 0 "C501" H 4700 2200 50  0000 L CNN
 F 1 "10uF" H 4700 2000 50  0000 L CNN
 F 2 "Capacitor_SMD:C_0603_1608Metric_Pad0.84x1.00mm_HandSolder" H 4700 2100 50  0001 C CNN
@@
 AR Path="/5AE473C8/5AE4BC4C" Ref="C516"  Part="1"
 AR Path="/5AF0307C/5AE4BC4C" Ref="C916"  Part="1"
-F 0 "C916" H 7600 1200 50  0000 L CNN
+F 0 "C516" H 7600 1200 50  0000 L CNN
 F 1 "100nF" H 7600 1000 50  0000 L CNN
 F 2 "Capacitor_SMD:C_0603_1608Metric_Pad0.84x1.00mm_HandSolder" H 7600 1100 50  0001 C CNN
@@
 AR Path="/5AE473C8/5AE50FA7" Ref="C515"  Part="1"
 AR Path="/5AF0307C/5AE50FA7" Ref="C915"  Part="1"
-F 0 "C915" H 7300 1200 50  0000 L CNN
+F 0 "C515" H 7300 1200 50  0000 L CNN
 F 1 "100nF" H 7300 1000 50  0000 L CNN
 F 2 "Capacitor_SMD:C_0603_1608Metric_Pad0.84x1.00mm_HandSolder" H 7300 1100 50  0001 C CNN
@@
 AR Path="/5AE473C8/5AE50FE1" Ref="C513"  Part="1"
 AR Path="/5AF0307C/5AE50FE1" Ref="C913"  Part="1"
-F 0 "C913" H 7000 1200 50  0000 L CNN
+F 0 "C513" H 7000 1200 50  0000 L CNN
 F 1 "100nF" H 7000 1000 50  0000 L CNN
 F 2 "Capacitor_SMD:C_0603_1608Metric_Pad0.84x1.00mm_HandSolder" H 7000 1100 50  0001 C CNN
@@
 AR Path="/5AE473C8/5AE5101D" Ref="C511"  Part="1"
 AR Path="/5AF0307C/5AE5101D" Ref="C911"  Part="1"
-F 0 "C911" H 6700 1200 50  0000 L CNN
+F 0 "C511" H 6700 1200 50  0000 L CNN
 F 1 "100nF" H 6700 1000 50  0000 L CNN
 F 2 "Capacitor_SMD:C_0603_1608Metric_Pad0.84x1.00mm_HandSolder" H 6700 1100 50  0001 C CNN
@@
 AR Path="/5AE473C8/5AE5105B" Ref="C509"  Part="1"
 AR Path="/5AF0307C/5AE5105B" Ref="C909"  Part="1"
-F 0 "C909" H 6400 1200 50  0000 L CNN
+F 0 "C509" H 6400 1200 50  0000 L CNN
 F 1 "100nF" H 6400 1000 50  0000 L CNN
 F 2 "Capacitor_SMD:C_0603_1608Metric_Pad0.84x1.00mm_HandSolder" H 6400 1100 50  0001 C CNN
@@
 AR Path="/5AE473C8/5AE70A1B" Ref="C505"  Part="1"
 AR Path="/5AF0307C/5AE70A1B" Ref="C905"  Part="1"
-F 0 "C905" H 5492 10346 50  0000 L CNN
+F 0 "C505" H 5492 10346 50  0000 L CNN
 F 1 "10pF" H 5492 10255 50  0000 L CNN
 F 2 "Capacitor_SMD:C_0603_1608Metric_Pad0.84x1.00mm_HandSolder" H 5400 10300 50  0001 C CNN
@@
 AR Path="/5AE473C8/5AE70BDB" Ref="R501"  Part="1"
 AR Path="/5AF0307C/5AE70BDB" Ref="R901"  Part="1"
-F 0 "R901" H 5859 10346 50  0000 L CNN
+F 0 "R501" H 5859 10346 50  0000 L CNN
 F 1 "5.62K" H 5859 10255 50  0000 L CNN
 F 2 "Resistor_SMD:R_0603_1608Metric_Pad0.84x1.00mm_HandSolder" H 5800 10300 50  0001 C CNN
@@
 AR Path="/5AE473C8/5AE98243" Ref="C502"  Part="1"
 AR Path="/5AF0307C/5AE98243" Ref="C902"  Part="1"
-F 0 "C902" H 4942 10046 50  0000 L CNN
+F 0 "C502" H 4942 10046 50  0000 L CNN
 F 1 "100nF" H 4942 9955 50  0000 L CNN
 F 2 "Capacitor_SMD:C_0603_1608Metric_Pad0.84x1.00mm_HandSolder" H 4850 10000 50  0001 C CNN
@@
 AR Path="/5AE473C8/5AEB7A30" Ref="L501"  Part="1"
 AR Path="/5AF0307C/5AEB7A30" Ref="L901"  Part="1"
-F 0 "L901" V 3972 9800 50  0000 C CNN
+F 0 "L501" V 3972 9800 50  0000 C CNN
 F 1 "L" V 4063 9800 50  0000 C CNN
 F 2 "Inductor_SMD:L_0603_1608Metric_Pad0.84x1.00mm_HandSolder" H 4150 9800 50  0001 C CNN
@@
 AR Path="/5AE473C8/5ACBEA02" Ref="U501"  Part="1"
 AR Path="/5AF0307C/5ACBEA02" Ref="U901"  Part="1"
-F 0 "U901" H 6250 10650 50  0000 C CNN
+F 0 "U501" H 6250 10650 50  0000 C CNN
 F 1 "ATSAME70Q21A-AN" H 6550 2950 50  0000 C CNN
 F 2 "Package_QFP:LQFP-144_20x20mm_P0.5mm" H 7300 6800 50  0001 C CNN
@@
 AR Path="/5AE473C8/5AF7855D" Ref="D501"  Part="1"
 AR Path="/5AF0307C/5AF7855D" Ref="D901"  Part="1"
-F 0 "D901" H 4900 4333 50  0000 C CNN
+F 0 "D501" H 4900 4333 50  0000 C CNN
 F 1 "LED_ARGB" H 4900 4424 50  0000 C CNN
 F 2 "LED_SMD:LED_RGB_1210" H 4900 4750 50  0001 C CNN
@@
 AR Path="/5AE473C8/5AE7EA0D" Ref="TP502"  Part="1"
 AR Path="/5AF0307C/5AE7EA0D" Ref="TP902"  Part="1"
-F 0 "TP902" V 3300 9700 50  0000 C CNN
+F 0 "TP502" V 3300 9700 50  0000 C CNN
 F 1 "AFE0_AD1" V 3204 9774 50  0000 C CNN
-F 2 "TestPoint:TestPoint_Pad_1.5x1.5mm" H 3300 9700 50  0001 C CNN
+F 2 "TestPoint:TestPoint_Pad_1.0x1.0mm" H 3300 9700 50  0001 C CNN
 F 3 "~" H 3300 9700 50  0001 C CNN
 	1    3100 9700
@@
 AR Path="/5AE473C8/5AE7EBD0" Ref="TP501"  Part="1"
 AR Path="/5AF0307C/5AE7EBD0" Ref="TP901"  Part="1"
-F 0 "TP901" V 3300 9200 50  0000 L CNN
+F 0 "TP501" V 3300 9200 50  0000 L CNN
 F 1 "AFE0_AD0" V 3200 9200 50  0000 L CNN
-F 2 "TestPoint:TestPoint_Pad_1.5x1.5mm" H 3300 9300 50  0001 C CNN
+F 2 "TestPoint:TestPoint_Pad_1.0x1.0mm" H 3300 9300 50  0001 C CNN
 F 3 "~" H 3300 9300 50  0001 C CNN
 	1    3100 9300
@@
 AR Path="/5AE473C8/5AE7F482" Ref="TP503"  Part="1"
 AR Path="/5AF0307C/5AE7F482" Ref="TP903"  Part="1"
-F 0 "TP903" V 3300 10200 50  0000 R CNN
+F 0 "TP503" V 3300 10200 50  0000 R CNN
 F 1 "ADVREF" V 3200 10250 50  0000 R CNN
-F 2 "TestPoint:TestPoint_Pad_1.5x1.5mm" H 3300 10100 50  0001 C CNN
+F 2 "TestPoint:TestPoint_Pad_1.0x1.0mm" H 3300 10100 50  0001 C CNN
 F 3 "~" H 3300 10100 50  0001 C CNN
 	1    3100 10100

Commit message: Fixed many rules check errors and changed the footprint of test points
Connections:
- no-connect marks 3 -> 91
Changed lines of the file:
@@
 Wire Wire Line
 	4400 9800 4400 10100
+NoConn ~ 6000 3600
+NoConn ~ 6000 3700
+NoConn ~ 6000 3800
+NoConn ~ 6000 3900
+NoConn ~ 6000 4000
+NoConn ~ 6000 4100
+NoConn ~ 6000 4200
+NoConn ~ 6000 4300
+NoConn ~ 6000 4400
+NoConn ~ 6000 4500
+NoConn ~ 6000 4600
+NoConn ~ 8600 3600
+NoConn ~ 8600 3700
+NoConn ~ 8600 3800
+NoConn ~ 8600 3900
+NoConn ~ 8600 4000
+NoConn ~ 8600 4100
+NoConn ~ 8600 4200
+NoConn ~ 8600 4300
+NoConn ~ 8600 4400
+NoConn ~ 8600 4500
+NoConn ~ 8600 4600
+NoConn ~ 8600 4700
+NoConn ~ 8600 4800
+NoConn ~ 8600 4900
+NoConn ~ 8600 5000
+NoConn ~ 6000 5100
+NoConn ~ 6000 5200
+NoConn ~ 6000 5300
+NoConn ~ 6000 5400
+NoConn ~ 6000 5500
+NoConn ~ 6000 5600
+NoConn ~ 6000 5800
+NoConn ~ 8600 5100
+NoConn ~ 8600 5200
+NoConn ~ 8600 5300
+NoConn ~ 8600 5400
+NoConn ~ 8600 5500
+NoConn ~ 8600 5600
+NoConn ~ 8600 5700
+NoConn ~ 8600 5800
+NoConn ~ 8600 5900
+NoConn ~ 6000 6400
+NoConn ~ 6000 6500
+NoConn ~ 6000 6600
+NoConn ~ 6000 6700
+NoConn ~ 6000 6900
+NoConn ~ 6000 7100
+NoConn ~ 6000 7200
+NoConn ~ 6000 7300
+NoConn ~ 8600 6700
+NoConn ~ 8600 6900
+NoConn ~ 8600 7000
+NoConn ~ 8600 7100
+NoConn ~ 8600 7200
+NoConn ~ 8600 7300
+NoConn ~ 8600 7400
+NoConn ~ 8600 7500
+NoConn ~ 8600 7600
+NoConn ~ 8600 7700
+NoConn ~ 8600 7800
+NoConn ~ 8600 7900
+NoConn ~ 6000 7700
+NoConn ~ 6000 7800
+NoConn ~ 6000 7900
+NoConn ~ 6000 8600
+NoConn ~ 6000 8700
+NoConn ~ 6000 8900
+NoConn ~ 6000 9000
+NoConn ~ 6000 9400
+NoConn ~ 6000 9600
+NoConn ~ 8600 8000
+NoConn ~ 8600 8100
+NoConn ~ 8600 8200
+NoConn ~ 8600 8300
+NoConn ~ 8600 8400
+NoConn ~ 8600 8500
+NoConn ~ 8600 8600
+NoConn ~ 8600 8700
+NoConn ~ 8600 8800
+NoConn ~ 8600 9200
+NoConn ~ 8600 9300
+NoConn ~ 8600 9400
+NoConn ~ 8600 9500
+NoConn ~ 8600 9600
+NoConn ~ 8600 9700
+NoConn ~ 8600 9800
+NoConn ~ 8600 10000
 $EndSCHEMATC

Commit message: Added the jumper for the ground pads
Parts:
- added JP501: GPAD_JP, Jumper:SolderJumper-3_P1.3mm_Open_Pad1.0x1.5mm, symbol Jumper:Jumper_3_Open
- added TP504: GPAD, TestPoint:TestPoint_Pad_1.0x1.0mm, symbol Venus-256-rescue:Test_Point-Connector_Specialized
Connections:
- wire segments 168 -> 172
- no-connect marks 91 -> 90
Changed lines of the file:
@@
 NoConn ~ 6000 7300
 NoConn ~ 8600 6700
-NoConn ~ 8600 6900
 NoConn ~ 8600 7000
 NoConn ~ 8600 7100
@@
 NoConn ~ 8600 9800
 NoConn ~ 8600 10000
+$Comp
+L Jumper:Jumper_3_Open JP501
+U 1 1 5B10913A
+P 9850 6900
+AR Path="/5AE473C8/5B10913A" Ref="JP501"  Part="1"
+AR Path="/5AF0307C/5B10913A" Ref="JP901"  Part="1"
+F 0 "JP501" H 9850 7124 50  0000 C CNN
+F 1 "GPAD_JP" H 9850 7033 50  0000 C CNN
+F 2 "Jumper:SolderJumper-3_P1.3mm_Open_Pad1.0x1.5mm" H 9850 6900 50  0001 C CNN
+F 3 "~" H 9850 6900 50  0001 C CNN
+	1    9850 6900
+	1    0    0    -1
+$EndComp
+Wire Wire Line
+	8600 6900 9600 6900
+Wire Wire Line
+	9850 7050 9850 7200
+Text HLabel 10500 6900 2    50   Input ~ 0
+GND
+Wire Wire Line
+	10100 6900 10500 6900
+Wire Wire Line
+	10500 7200 9850 7200
+$Comp
+L Venus-256-rescue:Test_Point-Connector_Specialized TP504
+U 1 1 5B1555DD
+P 10500 7200
+AR Path="/5AE473C8/5B1555DD" Ref="TP504"  Part="1"
+AR Path="/5AF0307C/5B1555DD" Ref="TP904"  Part="1"
+F 0 "TP504" V 10700 7250 50  0000 L CNN
+F 1 "GPAD" V 10600 7250 50  0000 L CNN
+F 2 "TestPoint:TestPoint_Pad_1.0x1.0mm" H 10700 7200 50  0001 C CNN
+F 3 "~" H 10700 7200 50  0001 C CNN
+	1    10500 7200
+	0    1    -1   0
+$EndComp
 $EndSCHEMATC
