File: Hardware/Schematics/BBDProto06/Venus-256/CellMaster.sch (KiCad schematic (older format))
At the start: 25 parts, among them U501 ATSAME70Q21A-AN

Commit message: Added the big pads behind the sensors
Changed lines of the file:
@@
 AR Path="/5AE473C8/5AE1DB3B" Ref="C514"  Part="1"
 AR Path="/5AF0307C/5AE1DB3B" Ref="C914"  Part="1"
-F 0 "C514" H 7100 2200 50  0000 L CNN
+F 0 "C914" H 7100 2200 50  0000 L CNN
 F 1 "100nF" H 7100 2000 50  0000 L CNN
 F 2 "Capacitor_SMD:C_0603_1608Metric_Pad0.84x1.00mm_HandSolder" H 7100 2100 50  0001 C CNN
@@
 AR Path="/5AE473C8/5AE23144" Ref="C512"  Part="1"
 AR Path="/5AF0307C/5AE23144" Ref="C912"  Part="1"
-F 0 "C512" H 6800 2200 50  0000 L CNN
+F 0 "C912" H 6800 2200 50  0000 L CNN
 F 1 "100nF" H 6800 2000 50  0000 L CNN
 F 2 "Capacitor_SMD:C_0603_1608Metric_Pad0.84x1.00mm_HandSolder" H 6800 2100 50  0001 C CNN
@@
 AR Path="/5AE473C8/5AE23174" Ref="C510"  Part="1"
 AR Path="/5AF0307C/5AE23174" Ref="C910"  Part="1"
-F 0 "C510" H 6500 2200 50  0000 L CNN
+F 0 "C910" H 6500 2200 50  0000 L CNN
 F 1 "100nF" H 6500 2000 50  0000 L CNN
 F 2 "Capacitor_SMD:C_0603_1608Metric_Pad0.84x1.00mm_HandSolder" H 6500 2100 50  0001 C CNN
@@
 AR Path="/5AE473C8/5AE231A2" Ref="C508"  Part="1"
 AR Path="/5AF0307C/5AE231A2" Ref="C908"  Part="1"
-F 0 "C508" H 6200 2200 50  0000 L CNN
+F 0 "C908" H 6200 2200 50  0000 L CNN
 F 1 "100nF" H 6200 2000 50  0000 L CNN
 F 2 "Capacitor_SMD:C_0603_1608Metric_Pad0.84x1.00mm_HandSolder" H 6200 2100 50  0001 C CNN
@@
 AR Path="/5AE473C8/5AE231D6" Ref="C507"  Part="1"
 AR Path="/5AF0307C/5AE231D6" Ref="C907"  Part="1"
-F 0 "C507" H 5900 2200 50  0000 L CNN
+F 0 "C907" H 5900 2200 50  0000 L CNN
 F 1 "100nF" H 5900 2000 50  0000 L CNN
 F 2 "Capacitor_SMD:C_0603_1608Metric_Pad0.84x1.00mm_HandSolder" H 5900 2100 50  0001 C CNN
@@
 AR Path="/5AE473C8/5AE23204" Ref="C506"  Part="1"
 AR Path="/5AF0307C/5AE23204" Ref="C906"  Part="1"
-F 0 "C506" H 5600 2200 50  0000 L CNN
+F 0 "C906" H 5600 2200 50  0000 L CNN
 F 1 "100nF" H 5600 2000 50  0000 L CNN
 F 2 "Capacitor_SMD:C_0603_1608Metric_Pad0.84x1.00mm_HandSolder" H 5600 2100 50  0001 C CNN
@@
 AR Path="/5AE473C8/5AE23234" Ref="C504"  Part="1"
 AR Path="/5AF0307C/5AE23234" Ref="C904"  Part="1"
-F 0 "C504" H 5300 2200 50  0000 L CNN
+F 0 "C904" H 5300 2200 50  0000 L CNN
 F 1 "100nF" H 5300 2000 50  0000 L CNN
 F 2 "Capacitor_SMD:C_0603_1608Metric_Pad0.84x1.00mm_HandSolder" H 5300 2100 50  0001 C CNN
@@
 AR Path="/5AE473C8/5AE23266" Ref="C503"  Part="1"
 AR Path="/5AF0307C/5AE23266" Ref="C903"  Part="1"
-F 0 "C503" H 5000 2200 50  0000 L CNN
+F 0 "C903" H 5000 2200 50  0000 L CNN
 F 1 "100nF" H 5000 2000 50  0000 L CNN
 F 2 "Capacitor_SMD:C_0603_1608Metric_Pad0.84x1.00mm_HandSolder" H 5000 2100 50  0001 C CNN
@@
 AR Path="/5AE473C8/5AE2329A" Ref="C501"  Part="1"
 AR Path="/5AF0307C/5AE2329A" Ref="C901"  Part="1"
-F 0 "C501" H 4700 2200 50  0000 L CNN
+F 0 "C901" H 4700 2200 50  0000 L CNN
 F 1 "10uF" H 4700 2000 50  0000 L CNN
 F 2 "Capacitor_SMD:C_0603_1608Metric_Pad0.84x1.00mm_HandSolder" H 4700 2100 50  0001 C CNN
@@
 AR Path="/5AE473C8/5AE4BC4C" Ref="C516"  Part="1"
 AR Path="/5AF0307C/5AE4BC4C" Ref="C916"  Part="1"
-F 0 "C516" H 7600 1200 50  0000 L CNN
+F 0 "C916" H 7600 1200 50  0000 L CNN
 F 1 "100nF" H 7600 1000 50  0000 L CNN
 F 2 "Capacitor_SMD:C_0603_1608Metric_Pad0.84x1.00mm_HandSolder" H 7600 1100 50  0001 C CNN
@@
 AR Path="/5AE473C8/5AE50FA7" Ref="C515"  Part="1"
 AR Path="/5AF0307C/5AE50FA7" Ref="C915"  Part="1"
-F 0 "C515" H 7300 1200 50  0000 L CNN
+F 0 "C915" H 7300 1200 50  0000 L CNN
 F 1 "100nF" H 7300 1000 50  0000 L CNN
 F 2 "Capacitor_SMD:C_0603_1608Metric_Pad0.84x1.00mm_HandSolder" H 7300 1100 50  0001 C CNN
@@
 AR Path="/5AE473C8/5AE50FE1" Ref="C513"  Part="1"
 AR Path="/5AF0307C/5AE50FE1" Ref="C913"  Part="1"
-F 0 "C513" H 7000 1200 50  0000 L CNN
+F 0 "C913" H 7000 1200 50  0000 L CNN
 F 1 "100nF" H 7000 1000 50  0000 L CNN
 F 2 "Capacitor_SMD:C_0603_1608Metric_Pad0.84x1.00mm_HandSolder" H 7000 1100 50  0001 C CNN
@@
 AR Path="/5AE473C8/5AE5101D" Ref="C511"  Part="1"
 AR Path="/5AF0307C/5AE5101D" Ref="C911"  Part="1"
-F 0 "C511" H 6700 1200 50  0000 L CNN
+F 0 "C911" H 6700 1200 50  0000 L CNN
 F 1 "100nF" H 6700 1000 50  0000 L CNN
 F 2 "Capacitor_SMD:C_0603_1608Metric_Pad0.84x1.00mm_HandSolder" H 6700 1100 50  0001 C CNN
@@
 AR Path="/5AE473C8/5AE5105B" Ref="C509"  Part="1"
 AR Path="/5AF0307C/5AE5105B" Ref="C909"  Part="1"
-F 0 "C509" H 6400 1200 50  0000 L CNN
+F 0 "C909" H 6400 1200 50  0000 L CNN
 F 1 "100nF" H 6400 1000 50  0000 L CNN
 F 2 "Capacitor_SMD:C_0603_1608Metric_Pad0.84x1.00mm_HandSolder" H 6400 1100 50  0001 C CNN
@@
 AR Path="/5AE473C8/5AE70A1B" Ref="C505"  Part="1"
 AR Path="/5AF0307C/5AE70A1B" Ref="C905"  Part="1"
-F 0 "C505" H 5492 10346 50  0000 L CNN
+F 0 "C905" H 5492 10346 50  0000 L CNN
 F 1 "10pF" H 5492 10255 50  0000 L CNN
 F 2 "Capacitor_SMD:C_0603_1608Metric_Pad0.84x1.00mm_HandSolder" H 5400 10300 50  0001 C CNN
@@
 AR Path="/5AE473C8/5AE70BDB" Ref="R501"  Part="1"
 AR Path="/5AF0307C/5AE70BDB" Ref="R901"  Part="1"
-F 0 "R501" H 5859 10346 50  0000 L CNN
+F 0 "R901" H 5859 10346 50  0000 L CNN
 F 1 "5.62K" H 5859 10255 50  0000 L CNN
 F 2 "Resistor_SMD:R_0603_1608Metric_Pad0.84x1.00mm_HandSolder" H 5800 10300 50  0001 C CNN
@@
 AR Path="/5AE473C8/5AE98243" Ref="C502"  Part="1"
 AR Path="/5AF0307C/5AE98243" Ref="C902"  Part="1"
-F 0 "C502" H 4942 10046 50  0000 L CNN
+F 0 "C902" H 4942 10046 50  0000 L CNN
 F 1 "100nF" H 4942 9955 50  0000 L CNN
 F 2 "Capacitor_SMD:C_0603_1608Metric_Pad0.84x1.00mm_HandSolder" H 4850 10000 50  0001 C CNN
@@
 AR Path="/5AE473C8/5AEB7A30" Ref="L501"  Part="1"
 AR Path="/5AF0307C/5AEB7A30" Ref="L901"  Part="1"
-F 0 "L501" V 3972 9800 50  0000 C CNN
+F 0 "L901" V 3972 9800 50  0000 C CNN
 F 1 "L" V 4063 9800 50  0000 C CNN
 F 2 "Inductor_SMD:L_0603_1608Metric_Pad0.84x1.00mm_HandSolder" H 4150 9800 50  0001 C CNN
@@
 AR Path="/5AE473C8/5ACBEA02" Ref="U501"  Part="1"
 AR Path="/5AF0307C/5ACBEA02" Ref="U901"  Part="1"
-F 0 "U501" H 6250 10650 50  0000 C CNN
+F 0 "U901" H 6250 10650 50  0000 C CNN
 F 1 "ATSAME70Q21A-AN" H 6550 2950 50  0000 C CNN
 F 2 "Package_QFP:LQFP-144_20x20mm_P0.5mm" H 7300 6800 50  0001 C CNN
@@
 AR Path="/5AE473C8/5AF7855D" Ref="D501"  Part="1"
 AR Path="/5AF0307C/5AF7855D" Ref="D901"  Part="1"
-F 0 "D501" H 4900 4333 50  0000 C CNN
+F 0 "D901" H 4900 4333 50  0000 C CNN
 F 1 "LED_ARGB" H 4900 4424 50  0000 C CNN
 F 2 "LED_SMD:LED_RGB_1210" H 4900 4750 50  0001 C CNN
@@
 AR Path="/5AE473C8/5AE7EA0D" Ref="TP502"  Part="1"
 AR Path="/5AF0307C/5AE7EA0D" Ref="TP902"  Part="1"
-F 0 "TP502" V 3300 9700 50  0000 C CNN
+F 0 "TP902" V 3300 9700 50  0000 C CNN
 F 1 "AFE0_AD1" V 3204 9774 50  0000 C CNN
 F 2 "TestPoint:TestPoint_Pad_1.0x1.0mm" H 3300 9700 50  0001 C CNN
@@
 AR Path="/5AE473C8/5AE7EBD0" Ref="TP501"  Part="1"
 AR Path="/5AF0307C/5AE7EBD0" Ref="TP901"  Part="1"
-F 0 "TP501" V 3300 9200 50  0000 L CNN
+F 0 "TP901" V 3300 9200 50  0000 L CNN
 F 1 "AFE0_AD0" V 3200 9200 50  0000 L CNN
 F 2 "TestPoint:TestPoint_Pad_1.0x1.0mm" H 3300 9300 50  0001 C CNN
@@
 AR Path="/5AE473C8/5AE7F482" Ref="TP503"  Part="1"
 AR Path="/5AF0307C/5AE7F482" Ref="TP903"  Part="1"
-F 0 "TP503" V 3300 10200 50  0000 R CNN
+F 0 "TP903" V 3300 10200 50  0000 R CNN
 F 1 "ADVREF" V 3200 10250 50  0000 R CNN
 F 2 "TestPoint:TestPoint_Pad_1.0x1.0mm" H 3300 10100 50  0001 C CNN
@@
 AR Path="/5AE473C8/5B10913A" Ref="JP501"  Part="1"
 AR Path="/5AF0307C/5B10913A" Ref="JP901"  Part="1"
-F 0 "JP501" H 9850 7124 50  0000 C CNN
+F 0 "JP901" H 9850 7124 50  0000 C CNN
 F 1 "GPAD_JP" H 9850 7033 50  0000 C CNN
 F 2 "Jumper:SolderJumper-3_P1.3mm_Open_Pad1.0x1.5mm" H 9850 6900 50  0001 C CNN
@@
 AR Path="/5AE473C8/5B1555DD" Ref="TP504"  Part="1"
 AR Path="/5AF0307C/5B1555DD" Ref="TP904"  Part="1"
-F 0 "TP504" V 10700 7250 50  0000 L CNN
+F 0 "TP904" V 10700 7250 50  0000 L CNN
 F 1 "GPAD" V 10600 7250 50  0000 L CNN
 F 2 "TestPoint:TestPoint_Pad_1.0x1.0mm" H 10700 7200 50  0001 C CNN

Commit message: Switched around the ADC channels to make the PCB simpler
Changed lines of the file:
@@
 AR Path="/5AE473C8/5AE1DB3B" Ref="C514"  Part="1"
 AR Path="/5AF0307C/5AE1DB3B" Ref="C914"  Part="1"
-F 0 "C914" H 7100 2200 50  0000 L CNN
+F 0 "C514" H 7100 2200 50  0000 L CNN
 F 1 "100nF" H 7100 2000 50  0000 L CNN
 F 2 "Capacitor_SMD:C_0603_1608Metric_Pad0.84x1.00mm_HandSolder" H 7100 2100 50  0001 C CNN
@@
 AR Path="/5AE473C8/5AE23144" Ref="C512"  Part="1"
 AR Path="/5AF0307C/5AE23144" Ref="C912"  Part="1"
-F 0 "C912" H 6800 2200 50  0000 L CNN
+F 0 "C512" H 6800 2200 50  0000 L CNN
 F 1 "100nF" H 6800 2000 50  0000 L CNN
 F 2 "Capacitor_SMD:C_0603_1608Metric_Pad0.84x1.00mm_HandSolder" H 6800 2100 50  0001 C CNN
@@
 AR Path="/5AE473C8/5AE23174" Ref="C510"  Part="1"
 AR Path="/5AF0307C/5AE23174" Ref="C910"  Part="1"
-F 0 "C910" H 6500 2200 50  0000 L CNN
+F 0 "C510" H 6500 2200 50  0000 L CNN
 F 1 "100nF" H 6500 2000 50  0000 L CNN
 F 2 "Capacitor_SMD:C_0603_1608Metric_Pad0.84x1.00mm_HandSolder" H 6500 2100 50  0001 C CNN
@@
 AR Path="/5AE473C8/5AE231A2" Ref="C508"  Part="1"
 AR Path="/5AF0307C/5AE231A2" Ref="C908"  Part="1"
-F 0 "C908" H 6200 2200 50  0000 L CNN
+F 0 "C508" H 6200 2200 50  0000 L CNN
 F 1 "100nF" H 6200 2000 50  0000 L CNN
 F 2 "Capacitor_SMD:C_0603_1608Metric_Pad0.84x1.00mm_HandSolder" H 6200 2100 50  0001 C CNN
@@
 AR Path="/5AE473C8/5AE231D6" Ref="C507"  Part="1"
 AR Path="/5AF0307C/5AE231D6" Ref="C907"  Part="1"
-F 0 "C907" H 5900 2200 50  0000 L CNN
+F 0 "C507" H 5900 2200 50  0000 L CNN
 F 1 "100nF" H 5900 2000 50  0000 L CNN
 F 2 "Capacitor_SMD:C_0603_1608Metric_Pad0.84x1.00mm_HandSolder" H 5900 2100 50  0001 C CNN
@@
 AR Path="/5AE473C8/5AE23204" Ref="C506"  Part="1"
 AR Path="/5AF0307C/5AE23204" Ref="C906"  Part="1"
-F 0 "C906" H 5600 2200 50  0000 L CNN
+F 0 "C506" H 5600 2200 50  0000 L CNN
 F 1 "100nF" H 5600 2000 50  0000 L CNN
 F 2 "Capacitor_SMD:C_0603_1608Metric_Pad0.84x1.00mm_HandSolder" H 5600 2100 50  0001 C CNN
@@
 AR Path="/5AE473C8/5AE23234" Ref="C504"  Part="1"
 AR Path="/5AF0307C/5AE23234" Ref="C904"  Part="1"
-F 0 "C904" H 5300 2200 50  0000 L CNN
+F 0 "C504" H 5300 2200 50  0000 L CNN
 F 1 "100nF" H 5300 2000 50  0000 L CNN
 F 2 "Capacitor_SMD:C_0603_1608Metric_Pad0.84x1.00mm_HandSolder" H 5300 2100 50  0001 C CNN
@@
 AR Path="/5AE473C8/5AE23266" Ref="C503"  Part="1"
 AR Path="/5AF0307C/5AE23266" Ref="C903"  Part="1"
-F 0 "C903" H 5000 2200 50  0000 L CNN
+F 0 "C503" H 5000 2200 50  0000 L CNN
 F 1 "100nF" H 5000 2000 50  0000 L CNN
 F 2 "Capacitor_SMD:C_0603_1608Metric_Pad0.84x1.00mm_HandSolder" H 5000 2100 50  0001 C CNN
@@
 AR Path="/5AE473C8/5AE2329A" Ref="C501"  Part="1"
 AR Path="/5AF0307C/5AE2329A" Ref="C901"  Part="1"
-F 0 "C901" H 4700 2200 50  0000 L CNN
+F 0 "C501" H 4700 2200 50  0000 L CNN
 F 1 "10uF" H 4700 2000 50  0000 L CNN
 F 2 "Capacitor_SMD:C_0603_1608Metric_Pad0.84x1.00mm_HandSolder" H 4700 2100 50  0001 C CNN
@@
 AR Path="/5AE473C8/5AE4BC4C" Ref="C516"  Part="1"
 AR Path="/5AF0307C/5AE4BC4C" Ref="C916"  Part="1"
-F 0 "C916" H 7600 1200 50  0000 L CNN
+F 0 "C516" H 7600 1200 50  0000 L CNN
 F 1 "100nF" H 7600 1000 50  0000 L CNN
 F 2 "Capacitor_SMD:C_0603_1608Metric_Pad0.84x1.00mm_HandSolder" H 7600 1100 50  0001 C CNN
@@
 AR Path="/5AE473C8/5AE50FA7" Ref="C515"  Part="1"
 AR Path="/5AF0307C/5AE50FA7" Ref="C915"  Part="1"
-F 0 "C915" H 7300 1200 50  0000 L CNN
+F 0 "C515" H 7300 1200 50  0000 L CNN
 F 1 "100nF" H 7300 1000 50  0000 L CNN
 F 2 "Capacitor_SMD:C_0603_1608Metric_Pad0.84x1.00mm_HandSolder" H 7300 1100 50  0001 C CNN
@@
 AR Path="/5AE473C8/5AE50FE1" Ref="C513"  Part="1"
 AR Path="/5AF0307C/5AE50FE1" Ref="C913"  Part="1"
-F 0 "C913" H 7000 1200 50  0000 L CNN
+F 0 "C513" H 7000 1200 50  0000 L CNN
 F 1 "100nF" H 7000 1000 50  0000 L CNN
 F 2 "Capacitor_SMD:C_0603_1608Metric_Pad0.84x1.00mm_HandSolder" H 7000 1100 50  0001 C CNN
@@
 AR Path="/5AE473C8/5AE5101D" Ref="C511"  Part="1"
 AR Path="/5AF0307C/5AE5101D" Ref="C911"  Part="1"
-F 0 "C911" H 6700 1200 50  0000 L CNN
+F 0 "C511" H 6700 1200 50  0000 L CNN
 F 1 "100nF" H 6700 1000 50  0000 L CNN
 F 2 "Capacitor_SMD:C_0603_1608Metric_Pad0.84x1.00mm_HandSolder" H 6700 1100 50  0001 C CNN
@@
 AR Path="/5AE473C8/5AE5105B" Ref="C509"  Part="1"
 AR Path="/5AF0307C/5AE5105B" Ref="C909"  Part="1"
-F 0 "C909" H 6400 1200 50  0000 L CNN
+F 0 "C509" H 6400 1200 50  0000 L CNN
 F 1 "100nF" H 6400 1000 50  0000 L CNN
 F 2 "Capacitor_SMD:C_0603_1608Metric_Pad0.84x1.00mm_HandSolder" H 6400 1100 50  0001 C CNN
@@
 AR Path="/5AE473C8/5AE70A1B" Ref="C505"  Part="1"
 AR Path="/5AF0307C/5AE70A1B" Ref="C905"  Part="1"
-F 0 "C905" H 5492 10346 50  0000 L CNN
+F 0 "C505" H 5492 10346 50  0000 L CNN
 F 1 "10pF" H 5492 10255 50  0000 L CNN
 F 2 "Capacitor_SMD:C_0603_1608Metric_Pad0.84x1.00mm_HandSolder" H 5400 10300 50  0001 C CNN
@@
 AR Path="/5AE473C8/5AE70BDB" Ref="R501"  Part="1"
 AR Path="/5AF0307C/5AE70BDB" Ref="R901"  Part="1"
-F 0 "R901" H 5859 10346 50  0000 L CNN
+F 0 "R501" H 5859 10346 50  0000 L CNN
 F 1 "5.62K" H 5859 10255 50  0000 L CNN
 F 2 "Resistor_SMD:R_0603_1608Metric_Pad0.84x1.00mm_HandSolder" H 5800 10300 50  0001 C CNN
@@
 AR Path="/5AE473C8/5AE98243" Ref="C502"  Part="1"
 AR Path="/5AF0307C/5AE98243" Ref="C902"  Part="1"
-F 0 "C902" H 4942 10046 50  0000 L CNN
+F 0 "C502" H 4942 10046 50  0000 L CNN
 F 1 "100nF" H 4942 9955 50  0000 L CNN
 F 2 "Capacitor_SMD:C_0603_1608Metric_Pad0.84x1.00mm_HandSolder" H 4850 10000 50  0001 C CNN
@@
 AR Path="/5AE473C8/5AEB7A30" Ref="L501"  Part="1"
 AR Path="/5AF0307C/5AEB7A30" Ref="L901"  Part="1"
-F 0 "L901" V 3972 9800 50  0000 C CNN
+F 0 "L501" V 3972 9800 50  0000 C CNN
 F 1 "L" V 4063 9800 50  0000 C CNN
 F 2 "Inductor_SMD:L_0603_1608Metric_Pad0.84x1.00mm_HandSolder" H 4150 9800 50  0001 C CNN
@@
 AR Path="/5AE473C8/5ACBEA02" Ref="U501"  Part="1"
 AR Path="/5AF0307C/5ACBEA02" Ref="U901"  Part="1"
-F 0 "U901" H 6250 10650 50  0000 C CNN
+F 0 "U501" H 6250 10650 50  0000 C CNN
 F 1 "ATSAME70Q21A-AN" H 6550 2950 50  0000 C CNN
 F 2 "Package_QFP:LQFP-144_20x20mm_P0.5mm" H 7300 6800 50  0001 C CNN
@@
 AR Path="/5AE473C8/5AF7855D" Ref="D501"  Part="1"
 AR Path="/5AF0307C/5AF7855D" Ref="D901"  Part="1"
-F 0 "D901" H 4900 4333 50  0000 C CNN
+F 0 "D501" H 4900 4333 50  0000 C CNN
 F 1 "LED_ARGB" H 4900 4424 50  0000 C CNN
 F 2 "LED_SMD:LED_RGB_1210" H 4900 4750 50  0001 C CNN
@@
 AR Path="/5AE473C8/5AE7EA0D" Ref="TP502"  Part="1"
 AR Path="/5AF0307C/5AE7EA0D" Ref="TP902"  Part="1"
-F 0 "TP902" V 3300 9700 50  0000 C CNN
+F 0 "TP502" V 3300 9700 50  0000 C CNN
 F 1 "AFE0_AD1" V 3204 9774 50  0000 C CNN
 F 2 "TestPoint:TestPoint_Pad_1.0x1.0mm" H 3300 9700 50  0001 C CNN
@@
 AR Path="/5AE473C8/5AE7EBD0" Ref="TP501"  Part="1"
 AR Path="/5AF0307C/5AE7EBD0" Ref="TP901"  Part="1"
-F 0 "TP901" V 3300 9200 50  0000 L CNN
+F 0 "TP501" V 3300 9200 50  0000 L CNN
 F 1 "AFE0_AD0" V 3200 9200 50  0000 L CNN
 F 2 "TestPoint:TestPoint_Pad_1.0x1.0mm" H 3300 9300 50  0001 C CNN
@@
 AR Path="/5AE473C8/5AE7F482" Ref="TP503"  Part="1"
 AR Path="/5AF0307C/5AE7F482" Ref="TP903"  Part="1"
-F 0 "TP903" V 3300 10200 50  0000 R CNN
+F 0 "TP503" V 3300 10200 50  0000 R CNN
 F 1 "ADVREF" V 3200 10250 50  0000 R CNN
 F 2 "TestPoint:TestPoint_Pad_1.0x1.0mm" H 3300 10100 50  0001 C CNN
@@
 AR Path="/5AE473C8/5B10913A" Ref="JP501"  Part="1"
 AR Path="/5AF0307C/5B10913A" Ref="JP901"  Part="1"
-F 0 "JP901" H 9850 7124 50  0000 C CNN
+F 0 "JP501" H 9850 7124 50  0000 C CNN
 F 1 "GPAD_JP" H 9850 7033 50  0000 C CNN
 F 2 "Jumper:SolderJumper-3_P1.3mm_Open_Pad1.0x1.5mm" H 9850 6900 50  0001 C CNN
@@
 AR Path="/5AE473C8/5B1555DD" Ref="TP504"  Part="1"
 AR Path="/5AF0307C/5B1555DD" Ref="TP904"  Part="1"
-F 0 "TP904" V 10700 7250 50  0000 L CNN
+F 0 "TP504" V 10700 7250 50  0000 L CNN
 F 1 "GPAD" V 10600 7250 50  0000 L CNN
 F 2 "TestPoint:TestPoint_Pad_1.0x1.0mm" H 10700 7200 50  0001 C CNN
