File: Hardware/Schematics/BBDProto07/Mars-64/Mars-64/Mars-64.kicad_pcb (KiCad board)
At the start: 4 copper layers, 43.2 x 50.8 mm, 76 parts, among them J1 Conn_02x06_Top_Bottom, J101 Conn_Coaxial, J102 Conn_Coaxial, J2 Conn_02x06_Top_Bottom, U101 ADG731, U102 ADG731

Commit message: Created the mirrored Pmod socket to allow daisy-chaining
Parts:
- J2: footprint Connector_PinHeader_2.54mm:PinHeader_2x06_P2.54mm_Vertical_SMD -> Connector_PinHeader_2.54mm:PinHeader_2x06_P2.54mm_Vertical_SMD_mirrored
