File: Hardware/Schematics/BBDProto07/Mars-64/Mars-64/Mars-64.sch (KiCad schematic (older format))
At the start: 70 parts, among them J01 Conn_Coaxial_x2, J02 Conn_02x06_Top_Bottom, U101 ADG731, U102 ADG731

Commit message: Set footprints
Parts:
- removed J01: Conn_Coaxial_x2, symbol Connector:Conn_Coaxial_x2
- added J2, J3: Conn_Coaxial, Connector_Coaxial:SMA_Molex_73251-2200_Horizontal, symbol Connector:Conn_Coaxial
- J1: renamed from J02; footprint (none) -> Connector_PinHeader_2.54mm:PinHeader_2x06_P2.54mm_Vertical
- JP4: renamed from JP03; footprint (none) -> Connector_PinHeader_2.54mm:PinHeader_1x03_P2.54mm_Vertical
- TP101, TP102, TP103, TP104, TP105, TP106, TP107, TP108, TP109, TP110, TP111, TP112, TP113, TP114, TP115, TP116, TP117, TP118, TP119, TP120, TP121, TP122, TP123, TP124, TP125, TP126, TP127, TP128, TP129, TP130, TP131, TP132, TP201, TP202, TP203, TP204, TP205, TP206, TP207, TP208, TP209, TP210, TP211, TP212, TP213, TP214, TP215, TP216, TP217, TP218, TP219, TP220, TP221, TP222, TP223, TP224, TP225, TP226, TP227, TP228, TP229, TP230, TP231, TP232: footprint (none) -> TestPoint:TestPoint_Pad_4.0x4.0mm
- TPAGND101: renamed from TPAGND; footprint (none) -> TestPoint:TestPoint_Pad_4.0x4.0mm
Connections:
- wire segments 132 -> 134

Commit message: Added the mouting holes
Parts:
- added H1, H2, H3, H4: MountingHole, MountingHole:MountingHole_2.2mm_M2, symbol Mechanical:MountingHole
Changed lines of the file:
@@
 Wire Wire Line
 	9000 5700 10300 5700
+$Comp
+L Mechanical:MountingHole H1
+U 1 1 5E2B4EA5
+P 8900 1100
+F 0 "H1" H 9000 1100 50  0000 L CNN
+F 1 "MountingHole" H 9000 1055 50  0001 L CNN
+F 2 "MountingHole:MountingHole_2.2mm_M2" H 8900 1100 50  0001 C CNN
+F 3 "~" H 8900 1100 50  0001 C CNN
+	1    8900 1100
+	1    0    0    -1
+$EndComp
+$Comp
+L Mechanical:MountingHole H2
+U 1 1 5E2B5DA6
+P 9200 1100
+F 0 "H2" H 9300 1100 50  0000 L CNN
+F 1 "MountingHole" H 9300 1055 50  0001 L CNN
+F 2 "MountingHole:MountingHole_2.2mm_M2" H 9200 1100 50  0001 C CNN
+F 3 "~" H 9200 1100 50  0001 C CNN
+	1    9200 1100
+	1    0    0    -1
+$EndComp
+$Comp
+L Mechanical:MountingHole H3
+U 1 1 5E2B6620
+P 8900 1300
+F 0 "H3" H 9000 1300 50  0000 L CNN
+F 1 "MountingHole" H 9000 1255 50  0001 L CNN
+F 2 "MountingHole:MountingHole_2.2mm_M2" H 8900 1300 50  0001 C CNN
+F 3 "~" H 8900 1300 50  0001 C CNN
+	1    8900 1300
+	1    0    0    -1
+$EndComp
+$Comp
+L Mechanical:MountingHole H4
+U 1 1 5E2B679E
+P 9200 1300
+F 0 "H4" H 9300 1300 50  0000 L CNN
+F 1 "MountingHole" H 9300 1255 50  0001 L CNN
+F 2 "MountingHole:MountingHole_2.2mm_M2" H 9200 1300 50  0001 C CNN
+F 3 "~" H 9200 1300 50  0001 C CNN
+	1    9200 1300
+	1    0    0    -1
+$EndComp
 $EndSCHEMATC

Commit message: Designed the first version of Mars-64's PCB
Parts:
- added J2: Conn_02x06_Top_Bottom, Connector_PinHeader_2.54mm:PinHeader_2x06_P2.54mm_Vertical_SMD, symbol Connector_Generic:Conn_02x06_Top_Bottom
- J1: footprint Connector_PinHeader_2.54mm:PinHeader_2x06_P2.54mm_Vertical -> Connector_PinHeader_2.54mm:PinHeader_2x06_P2.54mm_Vertical_SMD
- J101: renamed from J2; footprint Connector_Coaxial:SMA_Molex_73251-2200_Horizontal -> Connector_Coaxial:SMA_Amphenol_132134-10_Vertical
- J102: renamed from J3; footprint Connector_Coaxial:SMA_Molex_73251-2200_Horizontal -> Connector_Coaxial:SMA_Amphenol_132134-10_Vertical
- JP4: footprint Connector_PinHeader_2.54mm:PinHeader_1x03_P2.54mm_Vertical -> Jumper:SolderJumper-3_P1.3mm_Bridged2Bar12_Pad1.0x1.5mm_NumberLabels
- TPAGND1: renamed from TPAGND101; footprint TestPoint:TestPoint_Pad_4.0x4.0mm -> TestPoint:TestPoint_Pad_1.0x1.0mm
Connections:
- wire segments 134 -> 149
- no-connect marks 2 -> 6

Commit message: Created the mirrored Pmod socket to allow daisy-chaining
Parts:
- J2: footprint Connector_PinHeader_2.54mm:PinHeader_2x06_P2.54mm_Vertical_SMD -> Connector_PinHeader_2.54mm:PinHeader_2x06_P2.54mm_Vertical_SMD_mirrored
Changed lines of the file:
@@
 F 0 "J2" H 9050 1417 50  0000 C CNN
 F 1 "Conn_02x06_Top_Bottom" H 9050 1326 50  0001 C CNN
-F 2 "Connector_PinHeader_2.54mm:PinHeader_2x06_P2.54mm_Vertical_SMD" H 9000 1000 50  0001 C CNN
+F 2 "Connector_PinHeader_2.54mm:PinHeader_2x06_P2.54mm_Vertical_SMD_mirrored" H 9000 1000 50  0001 C CNN
 F 3 "~" H 9000 1000 50  0001 C CNN
 	1    9000 1000
