File: Hardware/Schematics/BBDProto07/Mars-64/Mars-64.kicad_pcb (KiCad board)
At the start: 4 copper layers, 50.8 x 50.8 mm, 76 parts, among them J101 Conn_Coaxial, J102 Conn_Coaxial, U101 ADG731, U102 ADG731

Commit message: Filled the fill area on In1.Cu
Other:
- board text added: "BBD Mars-64 rev. A"
Changed lines of the file:
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@@
   (general
     (thickness 1.6)
-    (drawings 6)
+    (drawings 7)
     (tracks 910)
     (zones 0)
@@
   (layers
     (0 F.Cu signal)
-    (1 In1.Cu signal hide)
+    (1 In1.Cu signal)
     (2 In2.Cu signal)
     (31 B.Cu signal)
@@
     (35 F.Paste user)
     (36 B.SilkS user)
-    (37 F.SilkS user hide)
+    (37 F.SilkS user)
     (38 B.Mask user)
     (39 F.Mask user)
@@
     )
   )
+  (gr_text "BBD Mars-64 rev. A" (at 60.96 78.74) (layer B.SilkS)
+    (effects (font (size 1.5 1.5) (thickness 0.3)) (justify mirror))
+  )
   (dimension 50.8 (width 0.15) (layer Dwgs.User)
     (gr_text "50.800 mm" (at 92.74 55.88 270) (layer Dwgs.User)
@@
   (segment (start 75.565 58.42) (end 78.875002 58.42) (width 0.25) (layer B.Cu) (net 1))
   (segment (start 79.3853 59.0476) (end 79.375 58.928) (width 0.25) (layer B.Cu) (net 1))
-  (via blind (at 49.403 65.278) (size 0.8) (drill 0.4) (layers In2.Cu B.Cu) (net 44))
   (segment (start 54.4653 59.69) (end 58.17 63.3947) (width 0.25) (layer B.Cu) (net 2))
   (segment (start 58.17 63.3947) (end 58.17 64.4175) (width 0.25) (layer B.Cu) (net 2))
@@
   (segment (start 53.24241 66.83) (end 53.52 66.83) (width 0.25) (layer B.Cu) (net 43))
   (segment (start 40.6396 64.0884) (end 41.0413 64.4901) (width 0.25) (layer B.Cu) (net 43))
+  (via blind (at 49.403 65.278) (size 0.8) (drill 0.4) (layers In2.Cu B.Cu) (net 44))
   (via blind (at 58.42 58.42) (size 0.8) (layers F.Cu In2.Cu) (net 44))
   (segment (start 54.2575 67.33) (end 53.106 67.33) (width 0.25) (layer B.Cu) (net 44))
