File: Hardware/Schematics/BBDProto07/Mars-64/Mars-64.sch (KiCad schematic (older format))
At the start: 76 parts, among them J1 Conn_02x06_Top_Bottom, J101 Conn_Coaxial, J102 Conn_Coaxial, J2 Conn_02x06_Top_Bottom, U101 ADG731, U102 ADG731

Commit message: Moved the Mars-64 source one directory up
Parts:
- Pmod1: renamed from J1; footprint Connector_PinHeader_2.54mm:PinHeader_2x06_P2.54mm_Vertical_SMD -> Mars-64:PinHeader_2x06_P2.54mm_Vertical_SMD_TopBottom
- Pmod2: renamed from J2; footprint Connector_PinHeader_2.54mm:PinHeader_2x06_P2.54mm_Vertical_SMD_mirrored -> Mars-64:PinHeader_2x06_P2.54mm_Vertical_SMD_TopBottom_Mirrored
Changed lines of the file:
@@
 $EndComp
 $Comp
-L Connector_Generic:Conn_02x06_Top_Bottom J1
+L Connector_Generic:Conn_02x06_Top_Bottom Pmod1
 U 1 1 5E2AF0E4
 P 9000 2200
-F 0 "J1" H 9050 2617 50  0000 C CNN
+F 0 "Pmod1" H 9050 2617 50  0000 C CNN
 F 1 "Conn_02x06_Top_Bottom" H 9050 2526 50  0001 C CNN
-F 2 "Connector_PinHeader_2.54mm:PinHeader_2x06_P2.54mm_Vertical_SMD" H 9000 2200 50  0001 C CNN
+F 2 "Mars-64:PinHeader_2x06_P2.54mm_Vertical_SMD_TopBottom" H 9000 2200 50  0001 C CNN
 F 3 "~" H 9000 2200 50  0001 C CNN
 	1    9000 2200
@@
 $EndComp
 $Comp
-L Connector_Generic:Conn_02x06_Top_Bottom J2
+L Connector_Generic:Conn_02x06_Top_Bottom Pmod2
 U 1 1 5E2E85D1
 P 9000 1000
-F 0 "J2" H 9050 1417 50  0000 C CNN
+F 0 "Pmod2" H 9050 1417 50  0000 C CNN
 F 1 "Conn_02x06_Top_Bottom" H 9050 1326 50  0001 C CNN
-F 2 "Connector_PinHeader_2.54mm:PinHeader_2x06_P2.54mm_Vertical_SMD_mirrored" H 9000 1000 50  0001 C CNN
+F 2 "Mars-64:PinHeader_2x06_P2.54mm_Vertical_SMD_TopBottom_Mirrored" H 9000 1000 50  0001 C CNN
 F 3 "~" H 9000 1000 50  0001 C CNN
 	1    9000 1000

Commit message: Updated the ADG731 symbol
Parts:
- U101, U102: symbol Mars-64-rescue:ADG731-Analog_Switch -> Analog_Switch:ADG731
Connections:
- wire segments 149 -> 145

Commit message: Changed the position of the Pmod pads
Parts:
- renumbered Pmod2 to PmodF2, Pmod1 to PmodM1
Changed lines of the file:
@@
 $EndComp
 $Comp
-L Connector_Generic:Conn_02x06_Top_Bottom Pmod1
+L Connector_Generic:Conn_02x06_Top_Bottom PmodM1
 U 1 1 5E2AF0E4
 P 9000 2200
-F 0 "Pmod1" H 9050 2617 50  0000 C CNN
+F 0 "PmodM1" H 9050 2617 50  0000 C CNN
 F 1 "Conn_02x06_Top_Bottom" H 9050 2526 50  0001 C CNN
 F 2 "Mars-64:PinHeader_2x06_P2.54mm_Vertical_SMD_TopBottom" H 9000 2200 50  0001 C CNN
@@
 $EndComp
 $Comp
-L Connector_Generic:Conn_02x06_Top_Bottom Pmod2
+L Connector_Generic:Conn_02x06_Top_Bottom PmodF2
 U 1 1 5E2E85D1
 P 9000 1000
-F 0 "Pmod2" H 9050 1417 50  0000 C CNN
+F 0 "PmodF2" H 9050 1417 50  0000 C CNN
 F 1 "Conn_02x06_Top_Bottom" H 9050 1326 50  0001 C CNN
 F 2 "Mars-64:PinHeader_2x06_P2.54mm_Vertical_SMD_TopBottom_Mirrored" H 9000 1000 50  0001 C CNN

Commit message: Removed the EP from the footprint of the multiplexers
Parts:
- U101, U102: footprint Package_QFP:TQFP-48-1EP_7x7mm_P0.5mm_EP5x5mm -> Package_QFP:TQFP-48_7x7mm_P0.5mm
Changed lines of the file:
@@
 Title "Mars-64"
 Date "2020-01-23"
-Rev "A"
+Rev "B"
 Comp "Bio Balance Detector"
 Comment1 ""
@@
 F 0 "U101" H 3000 5950 50  0000 L CNN
 F 1 "ADG731" H 3000 5850 50  0000 L CNN
-F 2 "Package_QFP:TQFP-48-1EP_7x7mm_P0.5mm_EP5x5mm" H 3550 1950 50  0001 L CNN
+F 2 "Package_QFP:TQFP-48_7x7mm_P0.5mm" H 3550 1950 50  0001 L CNN
 F 3 "https://www.analog.com/media/en/technical-documentation/data-sheets/ADG725_731.pdf" H 3310 4300 50  0001 C CNN
 	1    3300 3900
@@
 F 0 "U102" H 6300 5950 50  0000 L CNN
 F 1 "ADG731" H 6300 5850 50  0000 L CNN
-F 2 "Package_QFP:TQFP-48-1EP_7x7mm_P0.5mm_EP5x5mm" H 6850 1950 50  0001 L CNN
+F 2 "Package_QFP:TQFP-48_7x7mm_P0.5mm" H 6850 1950 50  0001 L CNN
 F 3 "https://www.analog.com/media/en/technical-documentation/data-sheets/ADG725_731.pdf" H 6610 4300 50  0001 C CNN
 	1    6600 3900

Commit message: Added a VSS jumper
Parts:
- added JP5: SolderJumper_2_Bridged, symbol Jumper:SolderJumper_2_Bridged
Connections:
- wire segments 145 -> 154
- no-connect marks 6 -> 4

Commit message: Added footprint to JP5 (VSS jumper)
Parts:
- JP5: footprint (none) -> Jumper:SolderJumper-2_P1.3mm_Bridged_RoundedPad1.0x1.5mm
Changed lines of the file:
@@
 F 0 "JP5" H 3000 6313 50  0000 C CNN
 F 1 "SolderJumper_2_Bridged" H 3000 6314 50  0001 C CNN
-F 2 "" H 3000 6200 50  0001 C CNN
+F 2 "Jumper:SolderJumper-2_P1.3mm_Bridged_RoundedPad1.0x1.5mm" H 3000 6200 50  0001 C CNN
 F 3 "~" H 3000 6200 50  0001 C CNN
 	1    3000 6200

Commit message: Added two capacitors to stabilize VCC
Parts:
- added C1, C2: 100 nF, Capacitor_SMD:C_1206_3216Metric_Pad1.42x1.75mm_HandSolder, symbol Device:C_Small
Connections:
- wire segments 154 -> 160
Changed lines of the file:
@@
 L power:GND #PWR0106
 U 1 1 5E32D300
-P 9800 2900
-F 0 "#PWR0106" H 9800 2650 50  0001 C CNN
-F 1 "GND" H 9805 2727 50  0000 C CNN
-F 2 "" H 9800 2900 50  0001 C CNN
-F 3 "" H 9800 2900 50  0001 C CNN
-	1    9800 2900
+P 10100 2900
+F 0 "#PWR0106" H 10100 2650 50  0001 C CNN
+F 1 "GND" H 10105 2727 50  0000 C CNN
+F 2 "" H 10100 2900 50  0001 C CNN
+F 3 "" H 10100 2900 50  0001 C CNN
+	1    10100 2900
 	1    0    0    -1
 $EndComp
@@
 	8300 2400 8800 2400
 Wire Wire Line
-	9300 2400 9800 2400
-Wire Wire Line
-	9800 2400 9800 2900
+	9300 2400 10100 2400
+Wire Wire Line
+	10100 2400 10100 2800
 Wire Wire Line
 	9300 2300 10200 2300
@@
 L power:GND #PWR0109
 U 1 1 5E3AFAD2
-P 9800 1700
-F 0 "#PWR0109" H 9800 1450 50  0001 C CNN
-F 1 "GND" H 9805 1527 50  0000 C CNN
-F 2 "" H 9800 1700 50  0001 C CNN
-F 3 "" H 9800 1700 50  0001 C CNN
-	1    9800 1700
+P 10100 1700
+F 0 "#PWR0109" H 10100 1450 50  0001 C CNN
+F 1 "GND" H 10105 1527 50  0000 C CNN
+F 2 "" H 10100 1700 50  0001 C CNN
+F 3 "" H 10100 1700 50  0001 C CNN
+	1    10100 1700
 	1    0    0    -1
 $EndComp
@@
 	8300 1200 8300 1700
 Wire Wire Line
-	9300 1200 9800 1200
-Wire Wire Line
-	9800 1200 9800 1700
+	9300 1200 10100 1200
+Wire Wire Line
+	10100 1200 10100 1600
 Text Label 8400 1300 0    50   ~ 0
 VCC3V3
@@
 Wire Wire Line
 	6800 1300 7700 1300
+$Comp
+L Device:C_Small C1
+U 1 1 5E6BE398
+P 9900 1600
+F 0 "C1" V 9671 1600 50  0000 C CNN
+F 1 "100 nF" V 9762 1600 50  0000 C CNN
+F 2 "Capacitor_SMD:C_1206_3216Metric_Pad1.42x1.75mm_HandSolder" H 9900 1600 50  0001 C CNN
+F 3 "~" H 9900 1600 50  0001 C CNN
+	1    9900 1600
+	0    1    1    0
+$EndComp
+$Comp
+L Device:C_Small C2
+U 1 1 5E6DCCB1
+P 9900 2800
+F 0 "C2" V 9671 2800 50  0000 C CNN
+F 1 "100 nF" V 9762 2800 50  0000 C CNN
+F 2 "Capacitor_SMD:C_1206_3216Metric_Pad1.42x1.75mm_HandSolder" H 9900 2800 50  0001 C CNN
+F 3 "~" H 9900 2800 50  0001 C CNN
+	1    9900 2800
+	0    1    1    0
+$EndComp
+Wire Wire Line
+	9700 1600 9800 1600
+Connection ~ 9700 1600
+Wire Wire Line
+	10000 1600 10100 1600
+Connection ~ 10100 1600
+Wire Wire Line
+	10100 1600 10100 1700
+Wire Wire Line
+	9700 2800 9800 2800
+Connection ~ 9700 2800
+Wire Wire Line
+	10000 2800 10100 2800
+Connection ~ 10100 2800
+Wire Wire Line
+	10100 2800 10100 2900
 $EndSCHEMATC

Commit message: Fixed a few bugs on the PCB and changed the revision from D to E
Connections:
- net labels added: VSS
Changed lines of the file:
@@
 Sheet 1 1
 Title "Mars-64"
-Date "2020-02-28"
-Rev "C"
+Date "2020-05-10"
+Rev "E"
 Comp "Bio Balance Detector"
 Comment1 ""
@@
 Wire Wire Line
 	10100 2800 10100 2900
+Text Label 9400 2000 0    50   ~ 0
+VSS
+Text Label 9400 800  0    50   ~ 0
+VSS
 $EndSCHEMATC
